File: eagle/1_cpu_control.brd (EAGLE design)
At the start: 160 x 100 mm, 41 parts, among them IC1 74LS08N, IC10 74LS173N, IC11 74LS273N, IC12 74LS74N, IC13 74LS157N, IC14 74LS157N, IC2 74LS163, IC3 74LS163, IC4 74LS00N, IC5 74LS273N, IC6 74LS148N, IC7 74LS148N, IC8 74LS08N, IC9 74S32N

Commit message: All boards prepared for MMU extension
Parts:
- JP10: device pinhead:2X16 -> pinhead:2X18
- moved JP10 2.54 mm to (105.4, 6.99)
Connections:
- new net /FP: JP10.34
- new net /IO: JP10.35
- new net /NP_FAULT: IC7.3, JP10.36
- new net /WR_FAULT: IC7.2, JP10.33
- net +5V: no longer IC7.2, IC7.3
Routing:
- net /WR_FAULT: track 0.00 -> 65.4 mm, vias 0 -> 2
- net /NP_FAULT: track 0.00 -> 60.9 mm, vias 0 -> 2
- net +5V: track 845.5 -> 840.4 mm
- net FAULT: track 81.9 -> 80.0 mm
- net /FI: track 16.8 -> 16.0 mm
Changed lines of the file:
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@@
 <layer number="18" name="Vias" color="2" fill="1" visible="yes" active="yes"/>
 <layer number="19" name="Unrouted" color="6" fill="1" visible="yes" active="yes"/>
-<layer number="20" name="Dimension" color="15" fill="1" visible="yes" active="yes"/>
+<layer number="20" name="Dimension" color="15" fill="1" visible="no" active="yes"/>
 <layer number="21" name="tPlace" color="7" fill="1" visible="no" active="yes"/>
 <layer number="22" name="bPlace" color="7" fill="1" visible="no" active="yes"/>
@@
 <layer number="97" name="Info" color="7" fill="1" visible="no" active="no"/>
 <layer number="98" name="Guide" color="6" fill="1" visible="no" active="no"/>
-<layer number="100" name="crosshair" color="7" fill="1" visible="yes" active="yes"/>
+<layer number="100" name="crosshair" color="7" fill="1" visible="no" active="yes"/>
 <layer number="121" name="_tsilk" color="14" fill="1" visible="yes" active="yes"/>
-<layer number="122" name="_bsilk" color="14" fill="1" visible="yes" active="yes"/>
+<layer number="122" name="_bsilk" color="14" fill="1" visible="no" active="yes"/>
 </layers>
 <board>
@@
 <wire x1="-4.7625" y1="-9.525" x2="-4.7625" y2="0" width="0.2032" layer="100"/>
 <wire x1="-9.525" y1="-4.7625" x2="0" y2="-4.7625" width="0.2032" layer="100"/>
+<wire x1="87.63" y1="5.08" x2="86.995" y2="4.445" width="0.254" layer="121"/>
+<wire x1="85.725" y1="4.445" x2="86.995" y2="4.445" width="0.254" layer="121"/>
+<wire x1="85.725" y1="4.445" x2="85.09" y2="5.08" width="0.254" layer="121"/>
+<wire x1="85.09" y1="5.08" x2="84.455" y2="4.445" width="0.254" layer="121"/>
+<wire x1="83.185" y1="4.445" x2="84.455" y2="4.445" width="0.254" layer="121"/>
+<wire x1="83.185" y1="4.445" x2="82.55" y2="5.08" width="0.254" layer="121"/>
+<wire x1="82.55" y1="8.89" x2="83.185" y2="9.525" width="0.254" layer="121"/>
+<wire x1="84.455" y1="9.525" x2="83.185" y2="9.525" width="0.254" layer="121"/>
+<wire x1="84.455" y1="9.525" x2="85.09" y2="8.89" width="0.254" layer="121"/>
+<wire x1="85.09" y1="8.89" x2="85.725" y2="9.525" width="0.254" layer="121"/>
+<wire x1="86.995" y1="9.525" x2="85.725" y2="9.525" width="0.254" layer="121"/>
+<wire x1="86.995" y1="9.525" x2="87.63" y2="8.89" width="0.254" layer="121"/>
+<wire x1="85.09" y1="5.08" x2="85.09" y2="8.89" width="0.254" layer="121"/>
+<wire x1="82.55" y1="5.08" x2="82.55" y2="8.89" width="0.254" layer="121"/>
 </plain>
 <attributes>
@@
 <element name="JP3" library="pinhead" package="2X08" value="" x="6.0325" y="75.565" rot="R270"/>
 <element name="JP4" library="pinhead" package="2X08" value="" x="6.0325" y="24.765" rot="R270"/>
-<element name="JP10" library="pinhead" package="2X16" value="" x="107.95" y="6.985" rot="R180"/>
+<element name="JP10" library="pinhead" package="2X18" value="" x="105.41" y="6.985" rot="R180"/>
 <element name="JP8" library="pinhead" package="1X05" value="" x="13.0175" y="79.375" rot="R90"/>
 <element name="JP7" library="pinhead" package="1X09" value="" x="153.3525" y="49.8475" rot="R270"/>
@@
 <contactref element="IC12" pad="11"/>
 <contactref element="IC12" pad="12"/>
+<wire x1="63.5" y1="36.83" x2="55.88" y2="36.83" width="0" layer="19" extent="1-1"/>
 </signal>
 <signal name="+5V">
@@
 <contactref element="IC7" pad="13"/>
 <contactref element="IC7" pad="1"/>
-<contactref element="IC7" pad="2"/>
-<contactref element="IC7" pad="3"/>
 <contactref element="IC7" pad="10"/>
 <contactref element="IC5" pad="1"/>
@@
 <wire x1="61.2775" y1="77.47" x2="64.4525" y2="77.47" width="0.8128" layer="16"/>
 <wire x1="45.72" y1="36.83" x2="45.72" y2="44.45" width="0.4064" layer="16"/>
-<wire x1="45.72" y1="36.83" x2="48.26" y2="36.83" width="0.4064" layer="16"/>
-<wire x1="48.26" y1="36.83" x2="50.8" y2="36.83" width="0.4064" layer="16"/>
 <wire x1="45.72" y1="44.45" x2="45.72" y2="45.4025" width="0.4064" layer="16"/>
 <wire x1="45.72" y1="45.4025" x2="46.99" y2="46.6725" width="0.4064" layer="16"/>
@@
 <wire x1="87.63" y1="55.88" x2="87.63" y2="36.5125" width="0.4064" layer="1"/>
 <wire x1="87.63" y1="36.5125" x2="90.17" y2="33.9725" width="0.4064" layer="1"/>
-<wire x1="90.17" y1="33.9725" x2="90.17" y2="26.67" width="0.4064" layer="1"/>
+<wire x1="90.17" y1="33.9725" x2="90.17" y2="27.94" width="0.4064" layer="1"/>
 <via x="23.1775" y="29.5275" extent="1-16" drill="0.6096" diameter="1.27"/>
-<wire x1="60.96" y1="26.67" x2="63.8175" y2="29.5275" width="0.4064" layer="1"/>
-<wire x1="63.8175" y1="29.5275" x2="87.3125" y2="29.5275" width="0.4064" layer="1"/>
-<wire x1="87.3125" y1="29.5275" x2="90.17" y2="26.67" width="0.4064" layer="1"/>
+<wire x1="60.96" y1="26.67" x2="60.96" y2="27.94" width="0.4064" layer="1"/>
+<wire x1="60.96" y1="27.94" x2="61.9125" y2="28.8925" width="0.4064" layer="1"/>
+<wire x1="61.9125" y1="28.8925" x2="89.2175" y2="28.8925" width="0.4064" layer="1"/>
+<wire x1="89.2175" y1="28.8925" x2="90.17" y2="27.94" width="0.4064" layer="1"/>
+<wire x1="90.17" y1="27.94" x2="90.17" y2="26.67" width="0.4064" layer="1"/>
 </signal>
 <signal name="N$3">
@@
 <wire x1="95.25" y1="19.05" x2="95.25" y2="17.4625" width="0.4064" layer="1"/>
 <wire x1="95.25" y1="17.4625" x2="94.615" y2="16.8275" width="0.4064" layer="1"/>
-<wire x1="94.615" y1="16.8275" x2="92.075" y2="16.8275" width="0.4064" layer="1"/>
-<wire x1="92.075" y1="16.8275" x2="91.44" y2="17.4625" width="0.4064" layer="1"/>
-<wire x1="91.44" y1="17.4625" x2="91.44" y2="20.6375" width="0.4064" layer="1"/>
-<wire x1="91.44" y1="20.6375" x2="90.17" y2="21.9075" width="0.4064" layer="1"/>
-<wire x1="62.5475" y1="21.9075" x2="90.17" y2="21.9075" width="0.4064" layer="1"/>
+<wire x1="94.615" y1="16.8275" x2="79.6925" y2="16.8275" width="0.4064" layer="1"/>
+<wire x1="79.6925" y1="16.8275" x2="74.6125" y2="21.9075" width="0.4064" layer="1"/>
+<wire x1="74.6125" y1="21.9075" x2="62.5475" y2="21.9075" width="0.4064" layer="1"/>
 </signal>
 <signal name="N$9">
@@
 <wire x1="120.65" y1="24.765" x2="121.92" y2="23.495" width="0.4064" layer="1"/>
 <wire x1="121.92" y1="23.495" x2="121.92" y2="19.05" width="0.4064" layer="1"/>
-<wire x1="113.03" y1="39.0525" x2="72.7075" y2="39.0525" width="0.4064" layer="16"/>
-<wire x1="72.7075" y1="39.0525" x2="70.1675" y2="41.5925" width="0.4064" layer="16"/>
-<wire x1="70.1675" y1="41.5925" x2="53.0225" y2="41.5925" width="0.4064" layer="16"/>
+<wire x1="113.03" y1="39.0525" x2="91.1225" y2="39.0525" width="0.4064" layer="16"/>
+<wire x1="91.1225" y1="39.0525" x2="88.5825" y2="41.5925" width="0.4064" layer="16"/>
+<wire x1="88.5825" y1="41.5925" x2="53.0225" y2="41.5925" width="0.4064" layer="16"/>
 </signal>
 <signal name="IRQ0">
@@
 <contactref element="IC9" pad="4"/>
 <contactref element="JP10" pad="32"/>
-<wire x1="92.71" y1="19.05" x2="92.71" y2="18.0975" width="0.4064" layer="16"/>
-<wire x1="92.71" y1="18.0975" x2="86.6775" y2="12.065" width="0.4064" layer="16"/>
-<wire x1="86.6775" y1="12.065" x2="86.6775" y2="7.9375" width="0.4064" layer="16"/>
-<wire x1="86.6775" y1="7.9375" x2="88.9" y2="5.715" width="0.4064" layer="16"/>
+<wire x1="88.9" y1="5.715" x2="87.63" y2="6.985" width="0.4064" layer="16"/>
+<wire x1="87.63" y1="6.985" x2="87.63" y2="13.0175" width="0.4064" layer="16"/>
+<wire x1="87.63" y1="13.0175" x2="92.71" y2="18.0975" width="0.4064" layer="16"/>
+<wire x1="92.71" y1="18.0975" x2="92.71" y2="19.05" width="0.4064" layer="16"/>
 </signal>
 <signal name="/FS">
@@
 <contactref element="JP10" pad="1"/>
 </signal>
+<signal name="/FP">
+<contactref element="JP10" pad="34"/>
+</signal>
+<signal name="/NP_FAULT">
+<contactref element="IC7" pad="3"/>
+<contactref element="JP10" pad="36"/>
+<wire x1="50.8" y1="36.83" x2="52.705" y2="38.735" width="0.4064" layer="16"/>
+<wire x1="52.705" y1="38.735" x2="73.66" y2="38.735" width="0.4064" layer="16"/>
+<wire x1="73.66" y1="38.735" x2="73.66" y2="30.1625" width="0.4064" layer="1"/>
+<wire x1="73.66" y1="30.1625" x2="76.5175" y2="27.305" width="0.4064" layer="16"/>
+<wire x1="76.5175" y1="27.305" x2="76.5175" y2="13.0175" width="0.4064" layer="16"/>
+<via x="73.66" y="38.735" extent="1-16" drill="0.6096"/>
+<via x="73.66" y="30.1625" extent="1-16" drill="0.6096"/>
+<wire x1="83.82" y1="5.715" x2="76.5175" y2="13.0175" width="0.4064" layer="16"/>
+</signal>
+<signal name="/WR_FAULT">
+<contactref element="IC7" pad="2"/>
+<contactref element="JP10" pad="33"/>
+<wire x1="48.26" y1="36.83" x2="51.435" y2="40.005" width="0.4064" layer="16"/>
+<wire x1="51.435" y1="40.005" x2="76.5175" y2="40.005" width="0.4064" layer="16"/>
+<wire x1="76.5175" y1="40.005" x2="76.5175" y2="30.1625" width="0.4064" layer="1"/>
+<wire x1="76.5175" y1="30.1625" x2="78.4225" y2="28.2575" width="0.4064" layer="16"/>
+<wire x1="78.4225" y1="28.2575" x2="78.4225" y2="16.1925" width="0.4064" layer="16"/>
+<via x="76.5175" y="40.005" extent="1-16" drill="0.6096"/>
+<via x="76.5175" y="30.1625" extent="1-16" drill="0.6096"/>
+<wire x1="86.36" y1="8.255" x2="78.4225" y2="16.1925" width="0.4064" layer="16"/>
+</signal>
+<signal name="/IO">
+<contactref element="JP10" pad="35"/>
+</signal>
 </signals>

Commit message: Removal of PPC started
Connections:
- removed net /LDPPC: IC11.11, IC12.3, IC9.11, JP10.11
- new net N$15: IC1.3, IC1.4
- new net N$17: IC11.11, IC12.3, IC9.11
- new net N$8: IC2.1, IC3.1
- net +5V: no longer IC1.4, IC1.5
- net /NEXTOP: now also IC1.6; no longer IC1.3, IC2.1, IC3.1
- net N$10: now also IC1.5
Routing:
- net /NEXTOP: track 134.8 -> 38.2 mm, vias 1 -> 0
- net /LDPPC: track 84.1 -> 0.00 mm, vias 1 -> 0
- net N$8: track 0.00 -> 16.3 mm
- net +5V: track 840.4 -> 830.2 mm
- net GND: track 16.5 -> 26.0 mm
Changed lines of the file:
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@@
 <contactref element="IC12" pad="11"/>
 <contactref element="IC12" pad="12"/>
-<wire x1="63.5" y1="36.83" x2="55.88" y2="36.83" width="0" layer="19" extent="1-1"/>
+<wire x1="55.88" y1="36.83" x2="58.1025" y2="34.6075" width="0.4064" layer="16"/>
+<wire x1="58.1025" y1="34.6075" x2="61.2775" y2="34.6075" width="0.4064" layer="16"/>
+<wire x1="61.2775" y1="34.6075" x2="63.5" y2="36.83" width="0.4064" layer="16"/>
 </signal>
 <signal name="+5V">
@@
 <contactref element="IC13" pad="16"/>
 <contactref element="C13" pad="1"/>
-<contactref element="IC1" pad="5"/>
-<contactref element="IC1" pad="4"/>
 <contactref element="IC4" pad="5"/>
 <contactref element="IC4" pad="1"/>
@@
 <wire x1="31.75" y1="47.3075" x2="31.75" y2="52.07" width="0.4064" layer="1"/>
 <wire x1="39.6875" y1="42.2275" x2="41.91" y2="44.45" width="0.8128" layer="16"/>
-<wire x1="55.88" y1="19.05" x2="55.88" y2="26.67" width="0.4064" layer="1"/>
-<wire x1="55.88" y1="26.67" x2="58.42" y2="26.67" width="0.4064" layer="1"/>
 <wire x1="53.34" y1="19.05" x2="55.88" y2="19.05" width="0.4064" layer="1"/>
 <wire x1="60.96" y1="19.05" x2="63.5" y2="19.05" width="0.4064" layer="1"/>
@@
 </signal>
 <signal name="/NEXTOP">
-<contactref element="IC2" pad="1"/>
-<contactref element="IC3" pad="1"/>
 <contactref element="IC10" pad="9"/>
 <contactref element="IC10" pad="10"/>
-<contactref element="IC1" pad="3"/>
 <contactref element="IC9" pad="12"/>
-<wire x1="16.51" y1="36.83" x2="15.24" y2="38.1" width="0.4064" layer="16"/>
-<wire x1="15.24" y1="38.1" x2="15.24" y2="50.8" width="0.4064" layer="16"/>
-<wire x1="15.24" y1="50.8" x2="16.51" y2="52.07" width="0.4064" layer="16"/>
-<wire x1="60.96" y1="26.67" x2="58.1025" y2="29.5275" width="0.4064" layer="16"/>
-<wire x1="58.1025" y1="29.5275" x2="23.1775" y2="29.5275" width="0.4064" layer="16"/>
-<wire x1="23.1775" y1="29.5275" x2="16.51" y2="36.195" width="0.4064" layer="1"/>
-<wire x1="16.51" y1="36.195" x2="16.51" y2="36.83" width="0.4064" layer="1"/>
 <wire x1="91.44" y1="59.69" x2="88.9" y2="59.69" width="0.4064" layer="1"/>
 <wire x1="91.44" y1="59.69" x2="87.63" y2="55.88" width="0.4064" layer="1"/>
 <wire x1="87.63" y1="55.88" x2="87.63" y2="36.5125" width="0.4064" layer="1"/>
 <wire x1="87.63" y1="36.5125" x2="90.17" y2="33.9725" width="0.4064" layer="1"/>
-<wire x1="90.17" y1="33.9725" x2="90.17" y2="27.94" width="0.4064" layer="1"/>
-<via x="23.1775" y="29.5275" extent="1-16" drill="0.6096" diameter="1.27"/>
-<wire x1="60.96" y1="26.67" x2="60.96" y2="27.94" width="0.4064" layer="1"/>
-<wire x1="60.96" y1="27.94" x2="61.9125" y2="28.8925" width="0.4064" layer="1"/>
-<wire x1="61.9125" y1="28.8925" x2="89.2175" y2="28.8925" width="0.4064" layer="1"/>
-<wire x1="89.2175" y1="28.8925" x2="90.17" y2="27.94" width="0.4064" layer="1"/>
-<wire x1="90.17" y1="27.94" x2="90.17" y2="26.67" width="0.4064" layer="1"/>
+<wire x1="90.17" y1="33.9725" x2="90.17" y2="26.67" width="0.4064" layer="1"/>
+<contactref element="IC1" pad="6"/>
+<wire x1="53.34" y1="26.67" x2="87.63" y2="36.5125" width="0" layer="19" extent="1-1"/>
 </signal>
 <signal name="N$3">
@@
 <wire x1="91.1225" y1="39.0525" x2="88.5825" y2="41.5925" width="0.4064" layer="16"/>
 <wire x1="88.5825" y1="41.5925" x2="53.0225" y2="41.5925" width="0.4064" layer="16"/>
+<contactref element="IC1" pad="5"/>
+<wire x1="55.88" y1="26.67" x2="53.0225" y2="41.5925" width="0" layer="19" extent="16-16"/>
 </signal>
 <signal name="IRQ0">
@@
 <wire x1="124.7775" y1="60.6425" x2="118.745" y2="66.675" width="0.4064" layer="16"/>
 <wire x1="118.745" y1="66.675" x2="109.22" y2="66.675" width="0.4064" layer="16"/>
-</signal>
-<signal name="/LDPPC">
-<contactref element="IC11" pad="11"/>
-<contactref element="IC12" pad="3"/>
-<contactref element="IC9" pad="11"/>
-<contactref element="JP10" pad="11"/>
-<wire x1="105.41" y1="52.3875" x2="108.9025" y2="55.88" width="0.4064" layer="16"/>
-<wire x1="108.9025" y1="55.88" x2="114.6175" y2="55.88" width="0.4064" layer="16"/>
-<wire x1="114.6175" y1="55.88" x2="118.4275" y2="59.69" width="0.4064" layer="16"/>
-<wire x1="118.4275" y1="59.69" x2="118.4275" y2="63.1825" width="0.4064" layer="1"/>
-<wire x1="118.4275" y1="63.1825" x2="116.205" y2="65.405" width="0.4064" layer="1"/>
-<wire x1="116.205" y1="65.405" x2="115.57" y2="65.405" width="0.4064" layer="1"/>
-<via x="118.4275" y="59.69" extent="1-16" drill="0.6096" diameter="1.27"/>
-<wire x1="92.71" y1="26.67" x2="92.71" y2="26.035" width="0.4064" layer="16"/>
-<wire x1="92.71" y1="26.035" x2="94.9325" y2="23.8125" width="0.4064" layer="16"/>
-<wire x1="94.9325" y1="23.8125" x2="99.06" y2="23.8125" width="0.4064" layer="16"/>
-<wire x1="99.06" y1="23.8125" x2="114.3" y2="8.5725" width="0.4064" layer="16"/>
-<wire x1="114.3" y1="8.5725" x2="114.3" y2="8.255" width="0.4064" layer="16"/>
-<wire x1="105.41" y1="51.7525" x2="92.71" y2="39.0525" width="0.4064" layer="1"/>
-<wire x1="92.71" y1="39.0525" x2="92.71" y2="26.67" width="0.4064" layer="1"/>
-<wire x1="105.41" y1="52.3875" x2="105.41" y2="52.07" width="0.4064" layer="16"/>
-<wire x1="105.41" y1="52.07" x2="105.41" y2="51.7525" width="0.4064" layer="1"/>
 </signal>
 <signal name="BUSCLKA">
@@
 <contactref element="JP10" pad="35"/>
 </signal>
+<signal name="N$8">
+<contactref element="IC2" pad="1"/>
+<contactref element="IC3" pad="1"/>
+<wire x1="16.51" y1="36.83" x2="15.24" y2="38.1" width="0.4064" layer="16"/>
+<wire x1="15.24" y1="38.1" x2="15.24" y2="50.8" width="0.4064" layer="16"/>
+<wire x1="15.24" y1="50.8" x2="16.51" y2="52.07" width="0.4064" layer="16"/>
+</signal>
+<signal name="N$15">
+<contactref element="IC1" pad="3"/>
+<contactref element="IC1" pad="4"/>
+<wire x1="58.42" y1="26.67" x2="60.96" y2="26.67" width="0" layer="19" extent="1-1"/>
+</signal>
+<signal name="N$17">
+<contactref element="IC9" pad="11"/>
+<contactref element="IC11" pad="11"/>
+<contactref element="IC12" pad="3"/>
+<wire x1="105.41" y1="52.07" x2="115.57" y2="65.405" width="0" layer="19" extent="1-1"/>
+<wire x1="92.71" y1="26.67" x2="105.41" y2="52.07" width="0" layer="19" extent="1-1"/>
+</signal>
 </signals>
