File: eagle/4_cpu_alu.brd (EAGLE design)
At the start: 160 x 100 mm, 33 parts, among them IC1 74LS181N, IC11 74LS244N, IC12 74LS244N, IC13 74LS244N, IC14 74LS244N, IC18 74LS04N, IC19 74LS32N, IC2 74LS181N, IC3 74LS181N, IC4 74LS181N, IC5 74S182N

Commit message: Removal of PPC started
Connections:
- removed net /LDPPC: JP10.11
Changed lines of the file:
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@@
 <?xml version="1.0" encoding="utf-8"?>
 <!DOCTYPE eagle SYSTEM "eagle.dtd">
-<eagle version="6.5.0">
+<eagle version="6.6.0">
 <drawing>
 <settings>
@@
 <contactref element="JP10" pad="1"/>
 </signal>
-<signal name="/LDPPC">
-<contactref element="JP10" pad="11"/>
-</signal>
 <signal name="BUSCLKA">
