File: eagle/4_cpu_alu.sch (EAGLE design)
At the start: 33 parts, among them IC1 74LS181N, IC11 74LS244N, IC12 74LS244N, IC13 74LS244N, IC14 74LS244N, IC18 74LS04N, IC19 74LS32N, IC2 74LS181N, IC3 74LS181N, IC4 74LS181N, IC5 74S182N

Commit message: Removal of PPC started
Connections:
- removed net /LDPPC: JP10.11
Changed lines of the file:
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@@
-</segment>
-</net>
-<net name="/LDPPC" class="0">
-<segment>
-<pinref part="JP10" gate="A" pin="11"/>
-<wire x1="83.82" y1="139.7" x2="73.66" y2="139.7" width="0.1524" layer="91"/>
-<label x="73.66" y="139.7" size="1.27" layer="95" rot="R180" xref="yes"/>
 </segment>
 </net>
