File: eagle/5_cpu_registers_a.sch (EAGLE design)
At the start: 43 parts, among them IC1 74LS374N, IC10 74LS374N, IC11 74LS374N, IC12 74LS374N, IC13 74LS374N, IC14 74LS374N, IC2 74LS374N, IC21 74LS08N, IC22 74LS32N, IC3 74LS374N, IC4 74LS374N, IC5 74LS374N, IC6 74LS374N, IC7 74LS374N, IC8 74LS374N, IC9 74LS374N

Commit message: Removal of PPC started
Parts:
- removed C7, C8: 100n, rcl:C-EU050-024X044
- removed IC7, IC8: 74LS374N, 74xx-eu:74LS374N
Connections:
- removed net /ENPPC: IC7A.OC, IC8A.OC, JP9.37
- removed net /LDPPC: IC7A.CLK, IC8A.CLK, JP10.11
- net +5V: no longer C7.1, C8.1, IC7P.VCC, IC8P.VCC
- net ABUS0: no longer IC7A.1D
- net ABUS1: no longer IC7A.2D
- net ABUS10: no longer IC8A.3D
- net ABUS11: no longer IC8A.4D
- net ABUS12: no longer IC8A.5D
- net ABUS13: no longer IC8A.6D
- net ABUS14: no longer IC8A.7D
- net ABUS15: no longer IC8A.8D
- net ABUS2: no longer IC7A.3D
- net ABUS3: no longer IC7A.4D
- net ABUS4: no longer IC7A.5D
- net ABUS5: no longer IC7A.6D
- net ABUS6: no longer IC7A.7D
- net ABUS7: no longer IC7A.8D
- net ABUS8: no longer IC8A.1D
- net ABUS9: no longer IC8A.2D
- net GND: no longer C7.2, C8.2, IC7P.GND, IC8P.GND
- net RBUS0: no longer IC7A.1Q
- net RBUS1: no longer IC7A.2Q
- net RBUS10: no longer IC8A.3Q
- net RBUS11: no longer IC8A.4Q
- net RBUS12: no longer IC8A.5Q
- net RBUS13: no longer IC8A.6Q
- net RBUS14: no longer IC8A.7Q
- net RBUS15: no longer IC8A.8Q
- net RBUS2: no longer IC7A.3Q
- net RBUS3: no longer IC7A.4Q
- net RBUS4: no longer IC7A.5Q
- net RBUS5: no longer IC7A.6Q
- net RBUS6: no longer IC7A.7Q
- net RBUS7: no longer IC7A.8Q
- net RBUS8: no longer IC8A.1Q
- net RBUS9: no longer IC8A.2Q
Other:
- note added: "(C) 2010-2016"
- note added: "2.0"
- note added: "Registers (MDR,DP,A,X,Y)"
- note removed: "(C) 2010-2014"
- note removed: "1.5"
- note removed: "Registers (MDR,DP,A,X,Y,PPC)"
- moved on the sheet: C17
