File: eagle/6_cpu_registers_b.brd (EAGLE design)
At the start: 160 x 100 mm, 47 parts, among them IC1 74LS569, IC10 74LS157N, IC11 74LS157N, IC12 74LS569, IC13 74LS569, IC14 74LS569, IC15 74LS569, IC16 74LS569, IC17 74LS569, IC18 74LS569, IC19 74LS569, IC2 74LS569, IC3 74LS569, IC4 74LS569, IC5 74LS569, IC6 74LS569, IC7 74LS569, IC8 74LS569, IC9 74LS08N

Commit message: Removal of PPC started
Connections:
- removed net /ENPPC: JP9.37
- removed net /LDPPC: JP10.11
Changed lines of the file:
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@@
 <contactref element="JP10" pad="14"/>
-</signal>
-<signal name="/LDPPC">
-<contactref element="JP10" pad="11"/>
 </signal>
 <signal name="BUSCLKA">
@@
 <contactref element="JP9" pad="41"/>
 </signal>
-<signal name="/ENPPC">
-<contactref element="JP9" pad="37"/>
-</signal>
 <signal name="/ENDP">
