File: eagle/6_cpu_registers_b.sch (EAGLE design)
At the start: 47 parts, among them IC1 74LS569, IC10 74LS157N, IC11 74LS157N, IC12 74LS569, IC13 74LS569, IC14 74LS569, IC15 74LS569, IC16 74LS569, IC17 74LS569, IC18 74LS569, IC19 74LS569, IC2 74LS569, IC3 74LS569, IC4 74LS569, IC5 74LS569, IC6 74LS569, IC7 74LS569, IC8 74LS569, IC9 74LS08N

Commit message: Removal of PPC started
Connections:
- removed net /ENPPC: JP9.37
- removed net /LDPPC: JP10.11
Changed lines of the file:
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@@
-</segment>
-</net>
-<net name="/LDPPC" class="0">
-<segment>
-<pinref part="JP10" gate="A" pin="11"/>
-<wire x1="83.82" y1="139.7" x2="73.66" y2="139.7" width="0.1524" layer="91"/>
-<label x="73.66" y="139.7" size="1.27" layer="95" rot="R180" xref="yes"/>
 </segment>
 </net>
@@
 </segment>
 </net>
-<net name="/ENPPC" class="0">
-<segment>
-<wire x1="83.82" y1="50.8" x2="73.66" y2="50.8" width="0.1524" layer="91"/>
-<pinref part="JP9" gate="A" pin="37"/>
-<label x="73.66" y="50.8" size="1.27" layer="95" rot="R180" xref="yes"/>
-</segment>
-</net>
