File: eagle/3_cpu_control.sch (EAGLE design)
At the start: 50 parts, among them IC1 74LS151N, IC10 74LS173N, IC11 74LS74N, IC12 74LS74N, IC13 74LS541N, IC14 74LS541N, IC15 74LS21N, IC16 74LS02N, IC17 74LS02N, IC18 74LS04N, IC2 74LS151N, IC20 74LS08N, IC3 74LS153N, IC4 74LS153N, IC5 74LS541N, IC6 74LS32N, IC7 74LS08N, IC8 74LS151N, IC9 74LS157N

Commit message: Renumbered boards and schematic sheets
Parts:
- removed C13, C14, C15, C16, C17, C18, C19: 100n, rcl:C-EU050-024X044
- removed C20: 10u, rcl:CPOL-EUE2.5-6
- removed IC10: 74LS173N, 74xx-eu:74LS173N
- removed IC11, IC12: 74LS74N, 74xx-eu:74LS74N
- removed IC13, IC14: 74LS541N, 74xx-us:74LS541N
- removed IC15: 74LS21N, 74xx-eu:74LS21N
- removed IC16, IC17: 74LS02N, 74xx-eu:74LS02N
- removed IC18: 74LS04N, 74xx-eu:74LS04N
- removed IC20, IC7: 74LS08N, 74xx-eu:74LS08N
- removed IC9: 74LS157N, 74xx-eu:74LS157N
- removed JP5: (no value), pinhead:PINHD-2X8
- added JP8: (no value), pinhead:PINHD-1X5
- added R1: 70, rcl:R-EU_0204/7
- added R10, R11, R12, R13, R14, R15, R16, R2, R3, R4, R5, R6, R7, R8, R9: (no value), rcl:R-EU_0204/7
- added UC1, UC2, UC3, UC4: AM29F020P, am29-memory:AM29F020P
- C12: value 100n -> 10u; device rcl:C-EU050-024X044 -> rcl:CPOL-EUE5-6
- IC1: value 74LS151N -> 74154N; device 74xx-eu:74LS151N -> 74xx-eu:74154N
- IC2: value 74LS151N -> 74LS139N; device 74xx-eu:74LS151N -> 74xx-eu:74LS139N
- IC3, IC4: value 74LS153N -> 74LS139N; device 74xx-eu:74LS153N -> 74xx-eu:74LS139N
- IC5: value 74LS541N -> 74LS00N; device 74xx-us:74LS541N -> 74xx-eu:74LS00N
- IC8: value 74LS151N -> 74LS08N; device 74xx-eu:74LS151N -> 74xx-eu:74LS08N
Connections:
- removed net ALU_C: IC1A.Y, IC9A.1B
- removed net ALU_N: IC3A.1Y, IC9A.3B
- removed net ALU_V: IC4A.1Y, IC9A.4B
- removed net ALU_Z: IC3A.2Y, IC9A.2B
- removed net F7: IC11A.Q, IC5A.A8
- removed net LBUS0: JP5.15
- removed net LBUS1: JP5.16
- removed net LBUS10: JP5.5
- removed net LBUS11: JP5.6
- removed net LBUS12: JP5.3
- removed net LBUS13: JP5.4
- removed net LBUS14: JP5.1
- removed net LBUS15: IC8A.C, JP5.2
- removed net LBUS2: JP5.13
- removed net LBUS3: JP5.14
- removed net LBUS4: JP5.11
- removed net LBUS5: JP5.12
- removed net LBUS6: JP5.9
- removed net LBUS7: IC2A.C, JP5.10
- removed net LBUS8: JP5.7
- removed net LBUS9: JP5.8
- removed net N$10: IC15B.I0, IC17A.O
- removed net N$11: IC15B.I1, IC17B.O
- removed net N$12: IC15B.I2, IC17C.O
- removed net N$13: IC15B.I3, IC17D.O
- removed net N$14: IC15A.O, IC20A.I0, IC3A.2C1
- removed net N$16: IC20A.O, IC3A.2C0
- removed net N$17: IC10A.G1, IC10A.G2, IC7D.O
- removed net N$19: IC2A.Y, IC4A.1C2
- removed net N$2: IC18B.O, IC1A.D6
- removed net N$21: IC18D.O, IC2A.D1, IC2A.D6, IC8A.D1, IC8A.D6
- removed net N$3: IC18A.O, IC1A.D4, IC1A.D5
- removed net N$32: IC10A.D1, IC9A.1Y
- removed net N$48: IC10A.D2, IC9A.2Y
- removed net N$49: IC10A.D3, IC9A.3Y
- removed net N$50: IC10A.D4, IC9A.4Y
- removed net N$51: IC7A.O, IC7D.I0
- removed net N$52: IC12A.CLK, IC6C.O
- removed net N$53: IC12B.CLK, IC6D.O
- removed net N$54: IC6C.I1, IC7B.O
- removed net N$55: IC6D.I1, IC7C.O
- removed net N$6: IC15A.I0, IC16A.O
- removed net N$7: IC15A.I1, IC16B.O
- removed net N$9: IC15A.I3, IC16D.O
- new net /CNT_SP: IC6D.I0, UC4G$1.D5
- new net /INC_PC: IC6C.I0, UC4G$1.D7
- new net /LATCH_NONE: IC4B.Y3, IC8B.I1
- new net ADDRBUS0: IC4A.A, UC1G$1.D1
- new net ADDRBUS1: IC4A.B, UC1G$1.D2
- new net BUSIFCMODE0: IC2B.A, IC4B.A, UC2G$1.D7
- new net BUSIFCMODE1: IC2B.B, IC4B.B, UC1G$1.D0
- new net CLBUS0: IC2A.A, UC1G$1.D6
- new net CLBUS1: IC2A.B, UC1G$1.D7
- new net CNT0: JP8.1, UC1G$1.A4, UC2G$1.A4, UC3G$1.A4, UC4G$1.A4
- new net CNT1: JP8.2, UC1G$1.A5, UC2G$1.A5, UC3G$1.A5, UC4G$1.A5
- new net CNT2: JP8.3, UC1G$1.A6, UC2G$1.A6, UC3G$1.A6, UC4G$1.A6
- new net CNT3: JP8.4, UC1G$1.A7, UC2G$1.A7, UC3G$1.A7, UC4G$1.A7
- new net CNT4: JP8.5, UC1G$1.A8, UC2G$1.A8, UC3G$1.A8, UC4G$1.A8
- new net CRBUS0: IC3A.A, UC1G$1.D3
- new net CRBUS1: IC3A.B, UC1G$1.D4
- new net LOAD0: IC1A.A, UC2G$1.D2
- new net LOAD1: IC1A.B, UC2G$1.D3
- new net LOAD2: IC1A.C, UC2G$1.D4
- new net LOAD3: IC1A.D, UC2G$1.D5
- new net N$31: IC1A.0, R1.1
- new net N$33: IC1A.1, R2.1
- new net N$34: IC1A.2, R3.1
- new net N$35: IC1A.3, R4.1
- new net N$36: IC1A.4, R5.1
- new net N$37: IC1A.5, R6.1
- new net N$38: IC1A.6, R7.1
- new net N$39: IC1A.7, R8.1
- new net N$40: IC1A.8, R9.1
- new net N$41: IC1A.9, R10.1
- new net N$42: IC1A.10, R11.1
- new net N$43: IC1A.11, R12.1
- new net N$44: IC1A.12, R13.1
- new net N$45: IC1A.13, R14.1
- new net N$56: IC1A.15, R16.1
- net +5V: now also C12.+, IC8A.I0, IC8A.I1, IC8C.I0, IC8C.I1, IC8D.I0, IC8D.I1, UC1G$1.!WE, UC1G$2.AVCC@1, UC2G$1.!WE, UC2G$2.AVCC@1, UC3G$1.!WE, UC3G$2.AVCC@1, UC4G$1.!WE, UC4G$2.AVCC@1; no longer C12.1, C13.1, C14.1, C15.1, C16.1, C17.1, C18.1, C19.1, C20.+, IC10P.VCC, IC11A.CLR, IC11A.PRE, IC11B.CLR, IC11P.VCC, IC12A.CLR, IC12B.PRE, IC12P.VCC, IC13P.VCC, IC14P.VCC, IC15P.VCC, IC16P.VCC, IC17P.VCC, IC18C.I, IC18E.I, IC18F.I, IC18P.VCC, IC20B.I0, IC20B.I1, IC20C.I0, IC20C.I1, IC20D.I0, IC20D.I1, IC20P.VCC, IC4A.2C0, IC4A.2C1, IC4A.2C2, IC4A.2C3, IC4A.2G, IC6A.I0, IC6A.I1, IC6B.I0, IC6B.I1, IC7P.VCC, IC9P.VCC
- net /ALUCARRYIN: now also UC3G$1.D3
- net /ALUHI2MEM: now also IC2B.Y3, IC5B.I1
- net /ALULO2MEM: now also IC2B.Y2, IC5B.I0
- net /ALUSHR: now also UC3G$1.D2; no longer IC1A.C
- net /BUSIFCEN: now also IC2B.G, IC8B.I0, UC2G$1.D6
- net /CARRY1: no longer IC18B.I
- net /CARRY3: no longer IC18A.I
- net /CNTSP: now also IC6D.O
- net /ENA: now also IC2A.Y1
- net /ENABUS: now also IC3A.Y2
- net /ENALU: now also IC6A.O
- net /ENDP: now also IC4A.Y2
- net /ENIPTR: now also IC3A.Y3; no longer IC13A.G1, IC13A.G2, IC14A.G1, IC14A.G2
- net /ENLMDR: now also IC2A.Y0
- net /ENMAR: now also IC4A.Y0
- net /ENMEM: now also IC6B.O
- net /ENMSW: now also IC3A.Y1; no longer IC5A.G1, IC5A.G2
- net /ENPC: now also IC4A.Y3
- net /ENRMDR: now also IC3A.Y0
- net /ENSP: now also IC4A.Y1
- net /ENX: now also IC2A.Y2
- net /ENY: now also IC2A.Y3
- net /FI: no longer IC12A.Q, IC5A.A5
- net /FP: no longer IC11B.Q, IC5A.A7
- net /FS: no longer IC12B.Q, IC5A.A6
- net /INCPC: now also IC6C.O
- net /INC_MAR: now also UC4G$1.D6
- net /LATCHFLAGS: now also IC4B.G
- net /LATCH_I: now also IC4B.Y0; no longer IC7B.I1
- net /LATCH_S: now also IC4B.Y1; no longer IC7C.I1
- net /LDA: now also R6.2
- net /LDAHI: now also R5.2
- net /LDALO: now also R4.2
- net /LDDP: now also R14.2
- net /LDMAR: now also R12.2
- net /LDMARHI: now also R11.2
- net /LDMARLO: now also R10.2
- net /LDMDR: now also R3.2
- net /LDMDRHI: now also R2.2
- net /LDMDRLO: now also R1.2
- net /LDMEM: now also R9.2
- net /LDMSW: now also R16.2; no longer IC11A.CLK, IC11B.CLK, IC7B.I0, IC7C.I0, IC7D.I1, IC9A.!A!/B
- net /LDPC: now also R15.2
- net /LDSP: now also R13.2
- net /LDX: now also R7.2
- net /LDY: now also R8.2
- net /LOAD_IR: now also UC2G$1.D1
- net /MEM2ALUHI: now also IC2B.Y1, IC5A.I1
- net /MEM2ALULO: now also IC2B.Y0, IC5A.I0
- net /RST: no longer IC11B.PRE, IC12A.PRE, IC12B.CLR
- net ALUBUS0: no longer IC17A.I0, IC9A.1A
- net ALUBUS1: no longer IC17A.I1, IC9A.2A
- net ALUBUS10: no longer IC16B.I0
- net ALUBUS11: no longer IC16B.I1
- net ALUBUS12: no longer IC16C.I0
- net ALUBUS13: no longer IC16C.I1
- net ALUBUS14: no longer IC16D.I0
- net ALUBUS15: no longer IC16D.I1, IC3A.1C0, IC3A.1C1, IC8A.A
- net ALUBUS2: no longer IC17B.I0, IC9A.3A
- net ALUBUS3: no longer IC17B.I1, IC9A.4A
- net ALUBUS4: no longer IC12A.D, IC17C.I0
- net ALUBUS5: no longer IC12B.D, IC17C.I1
- net ALUBUS6: no longer IC11B.D, IC17D.I0
- net ALUBUS7: no longer IC11A.D, IC17D.I1, IC2A.A, IC3A.1C2
- net ALUBUS8: no longer IC16A.I0
- net ALUBUS9: no longer IC16A.I1
- net ALUMODE: now also UC3G$1.D4
- net ALUOP0: now also UC3G$1.D5
- net ALUOP1: now also UC3G$1.D6; no longer IC18D.I, IC2A.D3, IC2A.D4, IC8A.D3, IC8A.D4
- net ALUOP2: now also UC3G$1.D7
- net ALUOP3: now also UC2G$1.D0
- net ALURES0: no longer IC1A.D0, IC1A.D2
- net ALURES8: no longer IC1A.D1
- net BUSCLKA: now also IC1A.G1
- net BUSCLKB: no longer IC6C.I0, IC6D.I0
- net CLK0D: now also IC6A.I1, IC6B.I1; no longer IC10A.CLK
- net FAULT: now also IC1A.G2, IC6C.I1, IC6D.I1
- net FC: now also UC1G$1.A3, UC2G$1.A3, UC3G$1.A3, UC4G$1.A3; no longer IC10A.Q1, IC5A.A1
- net FN: now also UC1G$1.A1, UC2G$1.A1, UC3G$1.A1, UC4G$1.A1; no longer IC10A.Q3, IC5A.A3
- net FV: now also UC1G$1.A0, UC2G$1.A0, UC3G$1.A0, UC4G$1.A0; no longer IC10A.Q4, IC5A.A4
- net FZ: now also UC1G$1.A2, UC2G$1.A2, UC3G$1.A2, UC4G$1.A2; no longer IC10A.Q2, IC5A.A2
- net GND: now also C12.-, IC3A.G, IC3B.A, IC3B.B, IC3B.G, IC4A.G, IC5C.I0, IC5C.I1, IC5D.I0, IC5D.I1, UC1G$1.!CE, UC1G$1.!OE, UC1G$2.AGND@1, UC2G$1.!CE, UC2G$1.!OE, UC2G$2.AGND@1, UC3G$1.!CE, UC3G$1.!OE, UC3G$2.AGND@1, UC4G$1.!CE, UC4G$1.!OE, UC4G$2.AGND@1; no longer C12.2, C13.2, C14.2, C15.2, C16.2, C17.2, C18.2, C19.2, C20.-, IC10A.M, IC10A.N, IC10P.GND, IC11P.GND, IC12P.GND, IC13A.A1, IC13A.A6, IC13A.A7, IC13A.A8, IC13P.GND, IC14A.A1, IC14A.A2, IC14A.A3, IC14A.A4, IC14A.A5, IC14A.A6, IC14A.A7, IC14A.A8, IC14P.GND, IC15P.GND, IC16P.GND, IC17P.GND, IC18P.GND, IC1A.D3, IC1A.D7, IC1A.G, IC20P.GND, IC2A.D0, IC2A.D2, IC2A.D5, IC2A.D7, IC3A.1C3, IC3A.1G, IC3A.2C3, IC3A.2G, IC4A.1C3, IC4A.1G, IC7P.GND, IC8A.D0, IC8A.D2, IC8A.D5, IC8A.D7, IC8A.G, IC9A.G, IC9P.GND
- net LOAD_FLAGS0: now also UC3G$1.D0; no longer IC1A.A, IC3A.A, IC4A.A, IC7A.I0
- net LOAD_FLAGS1: now also UC3G$1.D1; no longer IC1A.B, IC3A.B, IC4A.B, IC7A.I1
- net MDRLDINHBT: now also IC8B.O
- net MEMSEG: now also UC4G$1.D3
- net N$1: now also IC1A.14, R15.1; no longer IC4A.1C0, IC4A.1C1, IC8A.Y
- net N$15: now also IC5B.O, IC6B.I0; no longer IC15B.O, IC20A.I1, IC3A.2C2
- net N$8: now also IC5A.O, IC6A.I0; no longer IC15A.I2, IC16C.O
- net OP0: now also UC1G$1.A9, UC2G$1.A9, UC3G$1.A9, UC4G$1.A9; no longer IC13A.A2
- net OP1: now also UC1G$1.A10, UC2G$1.A10, UC3G$1.A10, UC4G$1.A10; no longer IC13A.A3
- net OP2: now also UC1G$1.A11, UC2G$1.A11, UC3G$1.A11, UC4G$1.A11; no longer IC13A.A4
- net OP3: now also UC1G$1.A12, UC2G$1.A12, UC3G$1.A12, UC4G$1.A12; no longer IC13A.A5
- net OP4: now also UC1G$1.A13, UC2G$1.A13, UC3G$1.A13, UC4G$1.A13
- net OP5: now also UC1G$1.A14, UC2G$1.A14, UC3G$1.A14, UC4G$1.A14
- net OP6: now also UC1G$1.A15, UC2G$1.A15, UC3G$1.A15, UC4G$1.A15
- net OP7: now also UC1G$1.A16, UC2G$1.A16, UC3G$1.A16, UC4G$1.A16
- net OP8: now also UC1G$1.A17, UC2G$1.A17, UC3G$1.A17, UC4G$1.A17
- net PROT: now also UC4G$1.D2
- net RBUS0: no longer IC13A.Y1, IC5A.Y1
- net RBUS1: no longer IC13A.Y2, IC5A.Y2
- net RBUS10: no longer IC14A.Y3
- net RBUS11: no longer IC14A.Y4
- net RBUS12: no longer IC14A.Y5
- net RBUS13: no longer IC14A.Y6
- net RBUS14: no longer IC14A.Y7
- net RBUS15: no longer IC14A.Y8, IC8A.B
- net RBUS2: no longer IC13A.Y3, IC5A.Y3
- net RBUS3: no longer IC13A.Y4, IC5A.Y4
- net RBUS4: no longer IC13A.Y5, IC5A.Y5
- net RBUS5: no longer IC13A.Y6, IC5A.Y6
- net RBUS6: no longer IC13A.Y7, IC5A.Y7
- net RBUS7: no longer IC13A.Y8, IC2A.B, IC5A.Y8
- net RBUS8: no longer IC14A.Y1
- net RBUS9: no longer IC14A.Y2
- net RST: no longer IC10A.CLR
- net SP_DIR: now also UC4G$1.D4
Other:
- note added: "(C) 2010-2016"
- note added: "CONTROL"
- note added: "CPU.2"
- note added: "Control (uROM, field decoders)"
- note removed: "(C) 2010-2014"
- note removed: "CPU.3"
- note removed: "Control (MSW, ALU flags)"

Commit message: Sat Feb  6 20:10:54 CET 2016
Connections:
- new net /IRET: UC4G$1.D0
- new net /MEMOP: UC4G$1.D1
Other:
- note added: "CPU.3"
- note removed: "CPU.2"
- moved on the sheet: IC1, IC2A, IC2B, IC5A, IC5B, IC6A, IC6B

Commit message: Mon Feb  8 16:27:58 CET 2016
Parts:
- JP8: device pinhead:PINHD-1X5 -> pinhead:PINHD-1X6
Connections:
- removed net /IRET: UC4G$1.D0
- new net /FRET: JP8.1, UC1G$1.D5
- net /MEMOP: now also JP10.11
- net CNT0: now also JP8.2; no longer JP8.1
- net CNT1: now also JP8.3; no longer JP8.2
- net CNT2: now also JP8.4; no longer JP8.3
- net CNT3: now also JP8.5; no longer JP8.4
- net CNT4: now also JP8.6; no longer JP8.5
Changed lines of the file:
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@@
 <part name="SUPPLY20" library="supply2" deviceset="GND" device=""/>
 <part name="SUPPLY21" library="supply2" deviceset="GND" device=""/>
-<part name="JP8" library="pinhead" deviceset="PINHD-1X5" device=""/>
+<part name="JP8" library="pinhead" deviceset="PINHD-1X6" device=""/>
 <part name="JP7" library="pinhead" deviceset="PINHD-1X9" device=""/>
 <part name="FRAME2" library="frames" deviceset="DINA3_L" device="" value="ABCD"/>
@@
 </segment>
 </net>
-<net name="/IRET" class="0">
+<net name="/FRET" class="0">
 <segment>
-<pinref part="UC4" gate="G$1" pin="D0"/>
-<wire x1="261.62" y1="88.9" x2="259.08" y2="86.36" width="0.1524" layer="91"/>
-<wire x1="259.08" y1="86.36" x2="246.38" y2="86.36" width="0.1524" layer="91"/>
-<label x="246.38" y="86.36" size="1.6764" layer="95"/>
+<pinref part="UC1" gate="G$1" pin="D5"/>
+<wire x1="86.36" y1="76.2" x2="83.82" y2="73.66" width="0.1524" layer="91"/>
+<wire x1="83.82" y1="73.66" x2="71.12" y2="73.66" width="0.1524" layer="91"/>
+<label x="71.12" y="73.66" size="1.6764" layer="95"/>
 </segment>
 </net>
@@
 <instance part="JP10" gate="A" x="86.36" y="132.08"/>
 <instance part="JP9" gate="A" x="86.36" y="68.58"/>
-<instance part="JP8" gate="A" x="144.78" y="147.32"/>
+<instance part="JP8" gate="A" x="142.24" y="144.78"/>
 <instance part="JP7" gate="A" x="167.64" y="142.24"/>
 </instances>
@@
 <net name="CNT0" class="0">
 <segment>
-<wire x1="142.24" y1="152.4" x2="134.62" y2="152.4" width="0.1524" layer="91"/>
-<label x="127" y="152.4" size="1.27" layer="95" xref="yes"/>
-<pinref part="JP8" gate="A" pin="1"/>
+<wire x1="139.7" y1="149.86" x2="132.08" y2="149.86" width="0.1524" layer="91"/>
+<label x="124.46" y="149.86" size="1.27" layer="95" xref="yes"/>
+<pinref part="JP8" gate="A" pin="2"/>
 </segment>
 </net>
 <net name="CNT1" class="0">
 <segment>
-<wire x1="142.24" y1="149.86" x2="134.62" y2="149.86" width="0.1524" layer="91"/>
-<label x="127" y="149.86" size="1.27" layer="95" xref="yes"/>
-<pinref part="JP8" gate="A" pin="2"/>
+<wire x1="139.7" y1="147.32" x2="132.08" y2="147.32" width="0.1524" layer="91"/>
+<label x="124.46" y="147.32" size="1.27" layer="95" xref="yes"/>
+<pinref part="JP8" gate="A" pin="3"/>
 </segment>
 </net>
 <net name="CNT2" class="0">
 <segment>
-<wire x1="142.24" y1="147.32" x2="134.62" y2="147.32" width="0.1524" layer="91"/>
-<label x="127" y="147.32" size="1.27" layer="95" xref="yes"/>
-<pinref part="JP8" gate="A" pin="3"/>
+<wire x1="139.7" y1="144.78" x2="132.08" y2="144.78" width="0.1524" layer="91"/>
+<label x="124.46" y="144.78" size="1.27" layer="95" xref="yes"/>
+<pinref part="JP8" gate="A" pin="4"/>
 </segment>
 </net>
 <net name="CNT3" class="0">
 <segment>
-<wire x1="142.24" y1="144.78" x2="134.62" y2="144.78" width="0.1524" layer="91"/>
-<label x="127" y="144.78" size="1.27" layer="95" xref="yes"/>
-<pinref part="JP8" gate="A" pin="4"/>
+<wire x1="139.7" y1="142.24" x2="132.08" y2="142.24" width="0.1524" layer="91"/>
+<label x="124.46" y="142.24" size="1.27" layer="95" xref="yes"/>
+<pinref part="JP8" gate="A" pin="5"/>
 </segment>
 </net>
 <net name="CNT4" class="0">
 <segment>
-<wire x1="142.24" y1="142.24" x2="134.62" y2="142.24" width="0.1524" layer="91"/>
-<label x="127" y="142.24" size="1.27" layer="95" xref="yes"/>
-<pinref part="JP8" gate="A" pin="5"/>
+<wire x1="139.7" y1="139.7" x2="132.08" y2="139.7" width="0.1524" layer="91"/>
+<label x="124.46" y="139.7" size="1.27" layer="95" xref="yes"/>
+<pinref part="JP8" gate="A" pin="6"/>
 </segment>
 </net>
@@
 </segment>
 </net>
+<net name="/MEMOP" class="0">
+<segment>
+<pinref part="JP10" gate="A" pin="11"/>
+<wire x1="83.82" y1="139.7" x2="73.66" y2="139.7" width="0.1524" layer="91"/>
+<label x="73.66" y="139.7" size="1.27" layer="95" rot="R180" xref="yes"/>
+</segment>
+</net>
+<net name="/FRET" class="0">
+<segment>
+<pinref part="JP8" gate="A" pin="1"/>
+<wire x1="139.7" y1="152.4" x2="132.08" y2="152.4" width="0.1524" layer="91"/>
+<label x="124.46" y="152.4" size="1.27" layer="95" xref="yes"/>
+</segment>
+</net>
