File: eagle/3_cpu_control.sch (EAGLE design)
At the start: 50 parts, among them IC1 74154N, IC2 74LS139N, IC3 74LS139N, IC4 74LS139N, IC5 74LS00N, IC6 74LS32N, IC8 74LS08N

Commit message: 2016-02-10 17:30 (completed boards 2,6,7)
Connections:
- removed net /ENPPC: JP9.37
Changed lines of the file:
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@@
-</segment>
-</net>
-<net name="/ENPPC" class="0">
-<segment>
-<wire x1="83.82" y1="50.8" x2="73.66" y2="50.8" width="0.1524" layer="91"/>
-<label x="73.66" y="50.8" size="1.27" layer="95" rot="R180" xref="yes"/>
-<pinref part="JP9" gate="A" pin="37"/>
 </segment>
 </net>

Commit message: Completed board 0
Changed lines of the file:
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@@
 <text x="289.56" y="27.94" size="2.54" layer="97" font="vector">Control (uROM, field decoders)</text>
 <text x="386.08" y="10.16" size="2.54" layer="97" font="vector" rot="R180">2.0</text>
-<text x="383.54" y="33.02" size="2.54" layer="97" font="vector" rot="R180">Dawid Pilawa</text>
-<text x="383.54" y="27.94" size="2.54" layer="97" font="vector" rot="R180">(C) 2010-2016</text>
+<text x="386.08" y="33.02" size="2.54" layer="97" font="vector" rot="R180">Dawid Pilawa</text>
+<text x="386.08" y="27.94" size="2.54" layer="97" font="vector" rot="R180">(C) 2010-2016</text>
 <text x="370.84" y="10.16" size="2.54" layer="97" font="vector" rot="R180">CPU.3</text>
 <text x="322.58" y="93.98" size="1.778" layer="95">CONTROL</text>
@@
 <text x="289.56" y="27.94" size="2.54" layer="97" font="vector">Control (uROM, field decoders)</text>
 <text x="386.08" y="10.16" size="2.54" layer="97" font="vector" rot="R180">2.0</text>
-<text x="383.54" y="33.02" size="2.54" layer="97" font="vector" rot="R180">Dawid Pilawa</text>
-<text x="383.54" y="27.94" size="2.54" layer="97" font="vector" rot="R180">(C) 2010-2016</text>
+<text x="386.08" y="33.02" size="2.54" layer="97" font="vector" rot="R180">Dawid Pilawa</text>
+<text x="386.08" y="27.94" size="2.54" layer="97" font="vector" rot="R180">(C) 2010-2016</text>
 <text x="370.84" y="10.16" size="2.54" layer="97" font="vector" rot="R180">CPU.3</text>
 <text x="10.16" y="246.38" size="6.4516" layer="91">BOARD CONNECTORS</text>
