File: eagle/2_cpu_control.sch (EAGLE design)
At the start: 50 parts, among them IC1 74154N, IC2 74LS139N, IC3 74LS138N, IC4 74LS139N, IC5 74LS00N, IC6 74LS32N, IC8 74LS08N

Commit message: All boards prepared for MMU extension
Parts:
- JP10: device pinhead:PINHD-2X16 -> pinhead:PINHD-2X18
Connections:
- new net /FP: JP10.34
- new net /IO: JP10.35
- new net /NP_FAULT: JP10.36
- new net /WR_FAULT: JP10.33
Other:
- note added: "2.0"
- note removed: "1.5"
Changed lines of the file:
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@@
 <part name="JP3" library="pinhead" deviceset="PINHD-2X8" device=""/>
 <part name="JP4" library="pinhead" deviceset="PINHD-2X8" device=""/>
-<part name="JP10" library="pinhead" deviceset="PINHD-2X16" device=""/>
+<part name="JP10" library="pinhead" deviceset="PINHD-2X18" device=""/>
 <part name="IC8" library="74xx-eu" deviceset="74*08" device="N" technology="LS"/>
 <part name="IC5" library="74xx-eu" deviceset="74*00" device="N" technology="LS"/>
@@
 <plain>
 <text x="289.56" y="27.94" size="2.54" layer="97" font="vector">Control (uROM, field decoders)</text>
-<text x="386.08" y="10.16" size="2.54" layer="97" font="vector" rot="R180">1.5</text>
+<text x="386.08" y="10.16" size="2.54" layer="97" font="vector" rot="R180">2.0</text>
 <text x="383.54" y="33.02" size="2.54" layer="97" font="vector" rot="R180">Dawid Pilawa</text>
 <text x="383.54" y="27.94" size="2.54" layer="97" font="vector" rot="R180">(C) 2010-2014</text>
@@
 <plain>
 <text x="289.56" y="27.94" size="2.54" layer="97" font="vector">Control (uROM, field decoders)</text>
-<text x="386.08" y="10.16" size="2.54" layer="97" font="vector" rot="R180">1.5</text>
+<text x="386.08" y="10.16" size="2.54" layer="97" font="vector" rot="R180">2.0</text>
 <text x="383.54" y="33.02" size="2.54" layer="97" font="vector" rot="R180">Dawid Pilawa</text>
 <text x="383.54" y="27.94" size="2.54" layer="97" font="vector" rot="R180">(C) 2010-2014</text>
@@
 <instance part="JP3" gate="A" x="154.94" y="226.06"/>
 <instance part="JP4" gate="A" x="154.94" y="187.96"/>
-<instance part="JP10" gate="A" x="86.36" y="134.62"/>
+<instance part="JP10" gate="A" x="86.36" y="132.08"/>
 <instance part="JP9" gate="A" x="86.36" y="68.58"/>
 <instance part="JP8" gate="A" x="144.78" y="147.32"/>
@@
 </segment>
 </net>
+<net name="/FP" class="0">
+<segment>
+<pinref part="JP10" gate="A" pin="34"/>
+<wire x1="91.44" y1="111.76" x2="101.6" y2="111.76" width="0.1524" layer="91"/>
+<label x="101.6" y="111.76" size="1.27" layer="95" xref="yes"/>
+</segment>
+</net>
+<net name="/WR_FAULT" class="0">
+<segment>
+<pinref part="JP10" gate="A" pin="33"/>
+<wire x1="83.82" y1="111.76" x2="73.66" y2="111.76" width="0.1524" layer="91"/>
+<label x="73.66" y="111.76" size="1.27" layer="95" rot="R180" xref="yes"/>
+</segment>
+</net>
+<net name="/NP_FAULT" class="0">
+<segment>
+<pinref part="JP10" gate="A" pin="36"/>
+<wire x1="91.44" y1="109.22" x2="101.6" y2="109.22" width="0.1524" layer="91"/>
+<label x="101.6" y="109.22" size="1.27" layer="95" xref="yes"/>
+</segment>
+</net>
+<net name="/IO" class="0">
+<segment>
+<pinref part="JP10" gate="A" pin="35"/>
+<wire x1="83.82" y1="109.22" x2="73.66" y2="109.22" width="0.1524" layer="91"/>
+<label x="73.66" y="109.22" size="1.27" layer="95" rot="R180" xref="yes"/>
+</segment>
+</net>

Commit message: Removal of PPC started
Connections:
- removed net /LDPPC: JP10.11
Changed lines of the file:
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@@
-</segment>
-</net>
-<net name="/LDPPC" class="0">
-<segment>
-<pinref part="JP10" gate="A" pin="11"/>
-<wire x1="83.82" y1="139.7" x2="73.66" y2="139.7" width="0.1524" layer="91"/>
-<label x="73.66" y="139.7" size="1.27" layer="95" rot="R180" xref="yes"/>
 </segment>
 </net>

Commit message: PPC removal completed, control card RBUS selector changed from LS138 to LS139, removed /LDPPC and /ENPPC signals
Parts:
- IC3: value 74LS138N -> 74LS139N; device 74xx-eu:74LS138N -> 74xx-eu:74LS139N
Connections:
- removed net CRBUS2: IC3A.C, UC1G$1.D5
- net +5V: no longer IC3A.G1
- net /ENPPC: no longer IC3A.Y4
- net GND: now also IC3A.G, IC3B.A, IC3B.B, IC3B.G; no longer IC3A.G2A, IC3A.G2B
Other:
- note added: "(C) 2010-2016"
- note removed: "(C) 2010-2014"
- moved on the sheet: IC4A, IC4B, IC8B

Commit message: Renumbered boards and schematic sheets
Parts:
- removed JP9: (no value), pinhead:PINHD-2X24
- removed R1: 70, rcl:R-EU_0204/7
- removed R10, R11, R12, R13, R14, R15, R16, R2, R3, R4, R5, R6, R7, R8, R9: (no value), rcl:R-EU_0204/7
- removed UC1, UC2, UC3, UC4: AM29F020P, am29-memory:AM29F020P
- added C13, C14: 100n, rcl:C-EU050-024X044
- added C15: 10u, rcl:CPOL-EUE5-6
- added IC10: 74LS173N, 74xx-eu:74LS173N
- added IC11: 74LS273N, 74xx-eu:74273N
- added IC12: 74LS74N, 74xx-eu:74LS74N
- added IC13, IC14: 74LS157N, 74xx-eu:74LS157N
- added IC7: 74LS148N, 74xx-eu:74LS148N
- added IC9: 74S32N, 74xx-eu:74S32N
- added JP1: (no value), pinhead:PINHD-2X8
- added RN1: 4.7k, resistor-sil:G08R
- C12: value 10u -> 100n; device rcl:CPOL-EUE5-6 -> rcl:C-EU050-024X044
- IC1: value 74154N -> 74LS08N; device 74xx-eu:74154N -> 74xx-eu:74LS08N
- IC2, IC3: value 74LS139N -> 74LS163; device 74xx-eu:74LS139N -> 74xx-eu:74160N
- IC4: value 74LS139N -> 74LS00N; device 74xx-eu:74LS139N -> 74xx-eu:74LS00N
- IC5: value 74LS00N -> 74LS273N; device 74xx-eu:74LS00N -> 74xx-eu:74273N
- IC6: value 74LS32N -> 74LS148N; device 74xx-eu:74LS32N -> 74xx-eu:74LS148N
Connections:
- removed net /ALUCARRYIN: JP9.2, UC3G$1.D3
- removed net /ALUSHR: JP9.1, UC3G$1.D2
- removed net /CARRY1: JP9.29
- removed net /CARRY3: JP9.31
- removed net /CNT_SP: IC6D.I0, UC4G$1.D5
- removed net /ENA: IC2A.Y1, JP9.33
- removed net /ENALU: IC6A.O, JP9.39
- removed net /ENDP: IC4A.Y2, JP9.44
- removed net /ENIPTR: IC3A.Y3, JP9.38
- removed net /ENLMDR: IC2A.Y0, JP9.34
- removed net /ENMAR: IC4A.Y0, JP9.48
- removed net /ENMSW: IC3A.Y1, JP9.40
- removed net /ENPC: IC4A.Y3, JP9.42
- removed net /ENPPC: JP9.37
- removed net /ENRMDR: IC3A.Y0, JP9.41
- removed net /ENSP: IC4A.Y1, JP9.46
- removed net /ENX: IC2A.Y2, JP9.36
- removed net /ENY: IC2A.Y3, JP9.35
- removed net /INC_MAR: JP9.32, UC4G$1.D6
- removed net /INC_PC: IC6C.I0, UC4G$1.D7
- removed net /LATCH_I: IC4B.Y0, JP9.47
- removed net /LATCH_NONE: IC4B.Y3, IC8B.I1
- removed net /LATCH_S: IC4B.Y1, JP9.45
- removed net /LDA: JP9.14, R6.2
- removed net /LDAHI: JP9.11, R5.2
- removed net /LDALO: JP9.12, R4.2
- removed net /LDDP: JP9.22, R14.2
- removed net /LDMAR: JP9.23, R12.2
- removed net /LDMARHI: JP9.17, R11.2
- removed net /LDMARLO: JP9.18, R10.2
- removed net /LDMDR: JP9.9, R3.2
- removed net /LDMDRHI: JP9.10, R2.2
- removed net /LDMDRLO: JP9.7, R1.2
- removed net /LDMSW: JP9.20, R16.2
- removed net /LDPC: JP9.19, R15.2
- removed net /LDSP: JP9.21, R13.2
- removed net /LDX: JP9.13, R7.2
- removed net /LDY: JP9.16, R8.2
- removed net ADDRBUS0: IC4A.A, UC1G$1.D1
- removed net ADDRBUS1: IC4A.B, UC1G$1.D2
- removed net ALUMODE: JP9.3, UC3G$1.D4
- removed net ALUOP0: JP9.4, UC3G$1.D5
- removed net ALUOP1: JP9.6, UC3G$1.D6
- removed net ALUOP2: JP9.5, UC3G$1.D7
- removed net ALUOP3: JP9.8, UC2G$1.D0
- removed net ALURES0: JP9.25
- removed net ALURES8: JP9.27
- removed net BUSIFCMODE0: IC2B.A, IC4B.A, UC2G$1.D7
- removed net BUSIFCMODE1: IC2B.B, IC4B.B, UC1G$1.D0
- removed net CLBUS0: IC2A.A, UC1G$1.D6
- removed net CLBUS1: IC2A.B, UC1G$1.D7
- removed net CRBUS0: IC3A.A, UC1G$1.D3
- removed net CRBUS1: IC3A.B, UC1G$1.D4
- removed net LOAD0: IC1A.A, UC2G$1.D2
- removed net LOAD1: IC1A.B, UC2G$1.D3
- removed net LOAD2: IC1A.C, UC2G$1.D4
- removed net LOAD3: IC1A.D, UC2G$1.D5
- removed net LOAD_FLAGS0: JP9.24, UC3G$1.D0
- removed net LOAD_FLAGS1: JP9.26, UC3G$1.D1
- removed net MDRLDINHBT: IC8B.O, JP9.43
- removed net N$31: IC1A.0, R1.1
- removed net N$33: IC1A.1, R2.1
- removed net N$34: IC1A.2, R3.1
- removed net N$35: IC1A.3, R4.1
- removed net N$36: IC1A.4, R5.1
- removed net N$37: IC1A.5, R6.1
- removed net N$38: IC1A.6, R7.1
- removed net N$39: IC1A.7, R8.1
- removed net N$40: IC1A.8, R9.1
- removed net N$41: IC1A.9, R10.1
- removed net N$42: IC1A.10, R11.1
- removed net N$43: IC1A.11, R12.1
- removed net N$44: IC1A.12, R13.1
- removed net N$45: IC1A.13, R14.1
- removed net N$56: IC1A.15, R16.1
- new net /FAULT_PF: IC4C.O, IC7A.7
- new net /NEXTOP: IC10A.G1, IC10A.G2, IC1B.O, IC9D.I0
- new net DBUS0: IC11A.D1, JP1.1
- new net DBUS1: IC11A.D2, JP1.3
- new net DBUS2: IC11A.D3, JP1.5
- new net DBUS3: IC11A.D4, JP1.7
- new net DBUS4: IC11A.D5, JP1.9
- new net DBUS5: IC11A.D6, JP1.11
- new net DBUS6: IC11A.D7, JP1.13
- new net DBUS7: IC11A.D8, JP1.15
- new net IRQ0: IC5A.D8, JP1.2, RN1.9
- new net IRQ1: IC5A.D7, JP1.4, RN1.8
- new net IRQ2: IC5A.D6, JP1.6, RN1.7
- new net IRQ3: IC5A.D5, JP1.8, RN1.6
- new net IRQ4: IC5A.D4, JP1.10, RN1.5
- new net IRQ5: IC5A.D3, JP1.12, RN1.4
- new net IRQ6: IC5A.D2, JP1.14, RN1.3
- new net IRQ7: IC5A.D1, JP1.16, RN1.2
- new net N$10: IC1B.I1, IC4D.I0, IC7A.GS, IC8D.I1
- new net N$11: IC10A.D1, IC8A.O
- new net N$12: IC10A.D2, IC8B.O
- new net N$13: IC10A.D3, IC8C.O
- new net N$14: IC12A.D, IC8D.O
- new net N$16: IC11A.Q2, IC13A.2B
- new net N$17: IC11A.CLK, IC12A.CLK, IC9D.O
- new net N$18: IC10A.Q1, IC13A.1A
- new net N$19: IC10A.Q2, IC13A.2A
- new net N$2: IC2A.RCO, IC3A.ENP, IC3A.ENT
- new net N$20: IC10A.Q3, IC13A.3A
- new net N$21: IC10A.Q4, IC13A.4A
- new net N$22: IC11A.Q8, IC14A.4B
- new net N$23: IC11A.Q7, IC14A.3B
- new net N$24: IC11A.Q6, IC14A.2B
- new net N$25: IC11A.Q5, IC14A.1B
- new net N$26: IC11A.Q1, IC13A.1B
- new net N$27: IC6A.EI, IC9B.O
- new net N$28: IC11A.Q3, IC13A.3B
- new net N$3: IC7A.A0, IC8A.I1
- new net N$30: IC11A.Q4, IC13A.4B
- new net N$4: IC6A.A1, IC8B.I0
- new net N$47: IC12A.Q, IC13A.!A!/B, IC14A.!A!/B
- new net N$5: IC7A.A1, IC8B.I1
- new net N$57: IC5A.Q8, IC6A.7
- new net N$58: IC5A.Q7, IC6A.6
- new net N$59: IC5A.Q6, IC6A.5
- new net N$6: IC7A.A2, IC8C.I1
- new net N$60: IC5A.Q5, IC6A.4
- new net N$61: IC5A.Q4, IC6A.3
- new net N$62: IC5A.Q3, IC6A.2
- new net N$63: IC5A.Q2, IC6A.1
- new net N$64: IC5A.Q1, IC6A.0
- new net N$7: IC6A.A2, IC8C.I0
- new net N$9: IC10A.D4, IC6A.GS, IC8D.I0
- net +5V: now also C12.1, C13.1, C14.1, C15.+, IC10P.VCC, IC11P.VCC, IC12A.CLR, IC12P.VCC, IC13P.VCC, IC14P.VCC, IC1C.I0, IC1C.I1, IC1D.I0, IC1D.I1, IC2A.ENP, IC2A.ENT, IC2A.LD, IC3A.LD, IC4A.I0, IC4A.I1, IC4B.I0, IC4B.I1, IC5A.CLR, IC7A.0, IC7A.1, IC7A.2, IC7A.3, IC7A.4, IC7P.VCC, IC9A.I0, IC9A.I1, IC9C.I0, IC9C.I1, IC9P.VCC, RN1.1; no longer C12.+, IC8A.I0, IC8A.I1, IC8C.I0, IC8C.I1, IC8D.I0, IC8D.I1, UC1G$1.!WE, UC1G$2.AVCC@1, UC2G$1.!WE, UC2G$2.AVCC@1, UC3G$1.!WE, UC3G$2.AVCC@1, UC4G$1.!WE, UC4G$2.AVCC@1
- net /ALUHI2MEM: no longer IC2B.Y3, IC5B.I1
- net /ALULO2MEM: no longer IC2B.Y2, IC5B.I0
- net /BUSIFCEN: now also IC4D.I1; no longer IC2B.G, IC8B.I0, UC2G$1.D6
- net /CNTSP: no longer IC6D.O
- net /ENABUS: no longer IC3A.Y2
- net /ENMEM: no longer IC6B.O
- net /FI: now also IC9B.I0
- net /FS: now also IC4C.I0
- net /INCPC: no longer IC6C.O
- net /LATCHFLAGS: now also IC4D.O; no longer IC4B.G
- net /LDMEM: no longer R9.2
- net /LOAD_IR: now also IC1A.I1; no longer UC2G$1.D1
- net /MEM2ALUHI: no longer IC2B.Y1, IC5A.I1
- net /MEM2ALULO: no longer IC2B.Y0, IC5A.I0
- net /NP_FAULT: now also IC7A.6
- net /RST: now also IC11A.CLR, IC12A.PRE, IC1A.I0
- net /WR_FAULT: now also IC7A.5
- net BUSCLKA: now also IC9D.I1; no longer IC1A.G1
- net CLK0A: now also IC10A.CLK, IC2A.CLK, IC3A.CLK, IC5A.CLK
- net CLK0D: no longer IC6A.I1, IC6B.I1
- net CNT0: now also IC2A.QA; no longer UC1G$1.A4, UC2G$1.A4, UC3G$1.A4, UC4G$1.A4
- net CNT1: now also IC2A.QB; no longer UC1G$1.A5, UC2G$1.A5, UC3G$1.A5, UC4G$1.A5
- net CNT2: now also IC2A.QC; no longer UC1G$1.A6, UC2G$1.A6, UC3G$1.A6, UC4G$1.A6
- net CNT3: now also IC2A.QD; no longer UC1G$1.A7, UC2G$1.A7, UC3G$1.A7, UC4G$1.A7
- net CNT4: now also IC3A.QA; no longer UC1G$1.A8, UC2G$1.A8, UC3G$1.A8, UC4G$1.A8
- net FAULT: now also IC7A.EO, IC9B.I1; no longer IC1A.G2, IC6C.I1, IC6D.I1
- net FC: no longer UC1G$1.A3, UC2G$1.A3, UC3G$1.A3, UC4G$1.A3
- net FN: no longer UC1G$1.A1, UC2G$1.A1, UC3G$1.A1, UC4G$1.A1
- net FV: no longer UC1G$1.A0, UC2G$1.A0, UC3G$1.A0, UC4G$1.A0
- net FZ: no longer UC1G$1.A2, UC2G$1.A2, UC3G$1.A2, UC4G$1.A2
- net GND: now also C12.2, C13.2, C14.2, C15.-, IC10A.M, IC10A.N, IC10P.GND, IC11P.GND, IC12B.CLK, IC12B.CLR, IC12B.D, IC12B.PRE, IC12P.GND, IC13A.G, IC13P.GND, IC14A.1A, IC14A.2A, IC14A.3A, IC14A.4A, IC14A.G, IC14P.GND, IC2A.A, IC2A.B, IC2A.C, IC2A.D, IC3A.A, IC3A.B, IC3A.C, IC3A.D, IC7A.EI, IC7P.GND, IC9P.GND; no longer C12.-, IC2A.G, IC3A.G, IC3B.A, IC3B.B, IC3B.G, IC4A.G, IC5C.I0, IC5C.I1, IC5D.I0, IC5D.I1, UC1G$1.!CE, UC1G$1.!OE, UC1G$2.AGND@1, UC2G$1.!CE, UC2G$1.!OE, UC2G$2.AGND@1, UC3G$1.!CE, UC3G$1.!OE, UC3G$2.AGND@1, UC4G$1.!CE, UC4G$1.!OE, UC4G$2.AGND@1
- net MEMSEG: no longer UC4G$1.D3
- net N$1: now also IC6A.A0, IC8A.I0; no longer IC1A.14, R15.1
- net N$15: now also IC1A.O, IC1B.I0; no longer IC5B.O, IC6B.I0
- net N$8: now also IC2A.CLR, IC3A.CLR; no longer IC5A.O, IC6A.I0
- net OP0: now also IC13A.1Y; no longer UC1G$1.A9, UC2G$1.A9, UC3G$1.A9, UC4G$1.A9
- net OP1: now also IC13A.2Y; no longer UC1G$1.A10, UC2G$1.A10, UC3G$1.A10, UC4G$1.A10
- net OP2: now also IC13A.3Y; no longer UC1G$1.A11, UC2G$1.A11, UC3G$1.A11, UC4G$1.A11
- net OP3: now also IC13A.4Y; no longer UC1G$1.A12, UC2G$1.A12, UC3G$1.A12, UC4G$1.A12
- net OP4: now also IC14A.1Y; no longer UC1G$1.A13, UC2G$1.A13, UC3G$1.A13, UC4G$1.A13
- net OP5: now also IC14A.2Y; no longer UC1G$1.A14, UC2G$1.A14, UC3G$1.A14, UC4G$1.A14
- net OP6: now also IC14A.3Y; no longer UC1G$1.A15, UC2G$1.A15, UC3G$1.A15, UC4G$1.A15
- net OP7: now also IC14A.4Y; no longer UC1G$1.A16, UC2G$1.A16, UC3G$1.A16, UC4G$1.A16
- net OP8: now also IC12A.!Q; no longer UC1G$1.A17, UC2G$1.A17, UC3G$1.A17, UC4G$1.A17
- net PROT: now also IC4C.I1; no longer UC4G$1.D2
- net RST: now also IC10A.CLR
- net SP_DIR: no longer UC4G$1.D4
Other:
- note added: "(C) 2010-2014"
- note added: "CPU.1"
- note added: "Control (ucode sequencer)"
- note removed: "(C) 2010-2016"
- note removed: "CONTROL"
- note removed: "CPU.2"
- note removed: "Control (uROM, field decoders)"
- moved on the sheet: C1, C10, C11, C2, C3, C4, C5, C6, C7, C8, C9, IC1P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

Commit message: Sat Feb  6 20:10:54 CET 2016
Other:
- note added: "CPU.2"
- note removed: "CPU.1"
Changed lines of the file:
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@@
 <text x="383.54" y="33.02" size="2.54" layer="97" font="vector" rot="R180">Dawid Pilawa</text>
 <text x="383.54" y="27.94" size="2.54" layer="97" font="vector" rot="R180">(C) 2010-2014</text>
-<text x="370.84" y="10.16" size="2.54" layer="97" font="vector" rot="R180">CPU.1</text>
+<text x="370.84" y="10.16" size="2.54" layer="97" font="vector" rot="R180">CPU.2</text>
 </plain>
 <instances>
@@
 <text x="383.54" y="33.02" size="2.54" layer="97" font="vector" rot="R180">Dawid Pilawa</text>
 <text x="383.54" y="27.94" size="2.54" layer="97" font="vector" rot="R180">(C) 2010-2014</text>
-<text x="370.84" y="10.16" size="2.54" layer="97" font="vector" rot="R180">CPU.1</text>
+<text x="370.84" y="10.16" size="2.54" layer="97" font="vector" rot="R180">CPU.2</text>
 <text x="10.16" y="246.38" size="6.4516" layer="91">BOARD CONNECTORS</text>
 </plain>

Commit message: Mon Feb  8 16:27:58 CET 2016
Parts:
- added IC15, IC16: 74LS163, 74xx-eu:74160N
- JP8: device pinhead:PINHD-1X5 -> pinhead:PINHD-1X6
Connections:
- removed net N$15: IC1A.O, IC1B.I0
- new net /FRET: IC2A.LD, IC3A.LD, JP8.1
- new net /MEMOP: JP10.11
- new net N$29: IC15A.QC, IC3A.C
- new net N$31: IC16A.QC, IC2A.C
- new net N$32: IC16A.QA, IC2A.A
- new net N$33: IC16A.QB, IC2A.B
- new net N$34: IC16A.QD, IC2A.D
- new net N$35: IC15A.QA, IC3A.A
- new net N$36: IC15A.QB, IC3A.B
- new net N$37: IC15A.QD, IC3A.D
- net +5V: now also IC15A.CLR, IC16A.CLR; no longer IC2A.LD, IC3A.LD
- net /NEXTOP: now also IC2A.CLR, IC3A.CLR
- net CLK0A: now also IC15A.CLK, IC16A.CLK
- net CNT0: now also IC16A.A, JP8.2; no longer JP8.1
- net CNT1: now also IC16A.B, JP8.3; no longer JP8.2
- net CNT2: now also IC16A.C, JP8.4; no longer JP8.3
- net CNT3: now also IC16A.D, JP8.5; no longer JP8.4
- net CNT4: now also IC15A.A, JP8.6; no longer JP8.5
- net GND: now also IC15A.ENP, IC15A.ENT, IC16A.ENP, IC16A.ENT; no longer IC2A.A, IC2A.B, IC2A.C, IC2A.D, IC3A.A, IC3A.B, IC3A.C, IC3A.D
- net N$10: now also IC15A.LD, IC16A.LD, IC1B.I0; no longer IC1B.I1
- net N$8: now also IC1A.O, IC1B.I1; no longer IC2A.CLR, IC3A.CLR
Other:
- moved on the sheet: C1, C10, C11, C12, C13, C14, C15, C2, C3, C4, C5, C6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

Commit message: 2016-02-09 13:30
Parts:
- added C16, C17, C18: 100n, rcl:C-EU050-024X044
- added IC17: 74LS04N, 74xx-eu:74LS04N
Connections:
- new net N$15: IC17A.O, IC9C.I1
- new net N$38: IC2A.CLR, IC3A.CLR, IC9C.O
- net +5V: now also C16.1, C17.1, C18.1, IC15P.VCC, IC16P.VCC, IC17P.VCC; no longer IC9C.I0, IC9C.I1
- net /FRET: now also IC17A.I
- net /NEXTOP: now also IC9C.I0; no longer IC2A.CLR, IC3A.CLR
- net GND: now also C16.2, C17.2, C18.2, IC15P.GND, IC16P.GND, IC17B.I, IC17C.I, IC17D.I, IC17E.I, IC17F.I, IC17P.GND
Other:
- moved on the sheet: C1, C10, C11, C12, C13, C14, C15, C2, C3, C4, C5, C6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

Commit message: 2016-02-09 18:12
Connections:
- net GND: now also IC15A.B, IC15A.C, IC15A.D
Changed lines of the file:
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@@
 <pinref part="SUPPLY1" gate="GND" pin="GND"/>
 <pinref part="IC16" gate="A" pin="ENT"/>
-<wire x1="35.56" y1="203.2" x2="35.56" y2="167.64" width="0.1524" layer="91"/>
+<wire x1="35.56" y1="203.2" x2="35.56" y2="180.34" width="0.1524" layer="91"/>
+<wire x1="35.56" y1="180.34" x2="35.56" y2="177.8" width="0.1524" layer="91"/>
+<wire x1="35.56" y1="177.8" x2="35.56" y2="175.26" width="0.1524" layer="91"/>
+<wire x1="35.56" y1="175.26" x2="35.56" y2="167.64" width="0.1524" layer="91"/>
 <wire x1="35.56" y1="167.64" x2="35.56" y2="165.1" width="0.1524" layer="91"/>
 <wire x1="35.56" y1="165.1" x2="35.56" y2="157.48" width="0.1524" layer="91"/>
@@
 <junction x="35.56" y="167.64"/>
 <junction x="35.56" y="203.2"/>
+<pinref part="IC15" gate="A" pin="B"/>
+<wire x1="38.1" y1="180.34" x2="35.56" y2="180.34" width="0.1524" layer="91"/>
+<pinref part="IC15" gate="A" pin="C"/>
+<wire x1="38.1" y1="177.8" x2="35.56" y2="177.8" width="0.1524" layer="91"/>
+<pinref part="IC15" gate="A" pin="D"/>
+<wire x1="38.1" y1="175.26" x2="35.56" y2="175.26" width="0.1524" layer="91"/>
+<junction x="35.56" y="175.26"/>
+<junction x="35.56" y="177.8"/>
+<junction x="35.56" y="180.34"/>
 </segment>
 <segment>
