File: eagle/2_cpu_control.sch (EAGLE design)
At the start: 47 parts, among them IC1 74LS08N, IC10 74LS173N, IC11 74LS273N, IC12 74LS74N, IC13 74LS157N, IC14 74LS157N, IC15 74LS163, IC16 74LS163, IC17 74LS04N, IC2 74LS163, IC3 74LS163, IC4 74LS00N, IC5 74LS273N, IC6 74LS148N, IC7 74LS148N, IC8 74LS08N, IC9 74S32N

Commit message: 2016-02-10 17:30 (completed boards 2,6,7)
Other:
- note added: "(C) 2010-2016"
- note added: "Control (microcode sequencer)"
- note removed: "(C) 2010-2014"
- note removed: "Control (ucode sequencer)"
Changed lines of the file:
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@@
 <sheet>
 <plain>
-<text x="289.56" y="27.94" size="2.54" layer="97" font="vector">Control (ucode sequencer)</text>
+<text x="289.56" y="27.94" size="2.54" layer="97" font="vector">Control (microcode sequencer)</text>
 <text x="386.08" y="10.16" size="2.54" layer="97" font="vector" rot="R180">2.0</text>
 <text x="383.54" y="33.02" size="2.54" layer="97" font="vector" rot="R180">Dawid Pilawa</text>
-<text x="383.54" y="27.94" size="2.54" layer="97" font="vector" rot="R180">(C) 2010-2014</text>
+<text x="383.54" y="27.94" size="2.54" layer="97" font="vector" rot="R180">(C) 2010-2016</text>
 <text x="370.84" y="10.16" size="2.54" layer="97" font="vector" rot="R180">CPU.2</text>
 </plain>
@@
 <sheet>
 <plain>
-<text x="289.56" y="27.94" size="2.54" layer="97" font="vector">Control (ucode sequencer)</text>
+<text x="289.56" y="27.94" size="2.54" layer="97" font="vector">Control (microcode sequencer)</text>
 <text x="386.08" y="10.16" size="2.54" layer="97" font="vector" rot="R180">2.0</text>
 <text x="383.54" y="33.02" size="2.54" layer="97" font="vector" rot="R180">Dawid Pilawa</text>
-<text x="383.54" y="27.94" size="2.54" layer="97" font="vector" rot="R180">(C) 2010-2014</text>
+<text x="383.54" y="27.94" size="2.54" layer="97" font="vector" rot="R180">(C) 2010-2016</text>
 <text x="370.84" y="10.16" size="2.54" layer="97" font="vector" rot="R180">CPU.2</text>
 <text x="10.16" y="246.38" size="6.4516" layer="91">BOARD CONNECTORS</text>

Commit message: Wed Feb 10 22:17:37 CET 2016 (completed boards 5,4)
Parts:
- IC9: value 74S32N -> 74LS32N; device 74xx-eu:74S32N -> 74xx-eu:74LS32N
Changed lines of the file:
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@@
 <part name="SUPPLY5" library="supply2" deviceset="GND" device=""/>
 <part name="IC4" library="74xx-eu" deviceset="74*00" device="N" technology="LS"/>
-<part name="IC9" library="74xx-eu" deviceset="74*32" device="N" technology="S"/>
+<part name="IC9" library="74xx-eu" deviceset="74*32" device="N" technology="LS" value="74LS32N"/>
 <part name="SUPPLY18" library="supply2" deviceset="+5V" device=""/>
 <part name="RN1" library="resistor-sil" deviceset="G08R" device="" value="4.7k"/>

Commit message: Completed board 0
Changed lines of the file:
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@@
 <text x="289.56" y="27.94" size="2.54" layer="97" font="vector">Control (microcode sequencer)</text>
 <text x="386.08" y="10.16" size="2.54" layer="97" font="vector" rot="R180">2.0</text>
-<text x="383.54" y="33.02" size="2.54" layer="97" font="vector" rot="R180">Dawid Pilawa</text>
-<text x="383.54" y="27.94" size="2.54" layer="97" font="vector" rot="R180">(C) 2010-2016</text>
+<text x="386.08" y="33.02" size="2.54" layer="97" font="vector" rot="R180">Dawid Pilawa</text>
+<text x="386.08" y="27.94" size="2.54" layer="97" font="vector" rot="R180">(C) 2010-2016</text>
 <text x="370.84" y="10.16" size="2.54" layer="97" font="vector" rot="R180">CPU.2</text>
 </plain>
@@
 <text x="289.56" y="27.94" size="2.54" layer="97" font="vector">Control (microcode sequencer)</text>
 <text x="386.08" y="10.16" size="2.54" layer="97" font="vector" rot="R180">2.0</text>
-<text x="383.54" y="33.02" size="2.54" layer="97" font="vector" rot="R180">Dawid Pilawa</text>
-<text x="383.54" y="27.94" size="2.54" layer="97" font="vector" rot="R180">(C) 2010-2016</text>
+<text x="386.08" y="33.02" size="2.54" layer="97" font="vector" rot="R180">Dawid Pilawa</text>
+<text x="386.08" y="27.94" size="2.54" layer="97" font="vector" rot="R180">(C) 2010-2016</text>
 <text x="370.84" y="10.16" size="2.54" layer="97" font="vector" rot="R180">CPU.2</text>
 <text x="10.16" y="246.38" size="6.4516" layer="91">BOARD CONNECTORS</text>
