File: eagle/3_cpu_control.brd (EAGLE design)
At the start: 160 x 100 mm, 50 parts, among them IC1 74154N, IC2 74LS139N, IC3 74LS139N, IC4 74LS139N, IC5 74LS00N, IC6 74LS32N, IC8 74LS08N

Commit message: 2016-02-10 17:30 (completed boards 2,6,7)
Connections:
- removed net /ENPPC: JP9.37
Changed lines of the file:
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@@
 <via x="32.7025" y="31.75" extent="1-16" drill="0.6096"/>
-</signal>
-<signal name="/ENPPC">
-<contactref element="JP9" pad="37"/>
 </signal>
 <signal name="/ENMAR">
