File: eagle/3_cpu_control.brd (EAGLE design)
At the start: 160 x 100 mm, 50 parts, among them IC1 74154N, IC2 74LS139N, IC3 74LS139N, IC4 74LS139N, IC5 74LS00N, IC6 74LS32N, IC8 74LS08N

Commit message: Completed board 3
Routing:
- net /MEMOP: track 0.00 -> 59.2 mm, vias 0 -> 1
Other:
- board text added: "74LS154N"
- board text removed: "74154N"
Changed lines of the file:
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@@
 <layer number="21" name="tPlace" color="7" fill="1" visible="no" active="yes"/>
 <layer number="22" name="bPlace" color="7" fill="1" visible="no" active="yes"/>
-<layer number="23" name="tOrigins" color="15" fill="1" visible="yes" active="yes"/>
+<layer number="23" name="tOrigins" color="15" fill="1" visible="no" active="yes"/>
 <layer number="24" name="bOrigins" color="15" fill="1" visible="no" active="yes"/>
 <layer number="25" name="tNames" color="7" fill="1" visible="no" active="yes"/>
@@
 <wire x1="84.074" y1="19.177" x2="84.074" y2="49.403" width="0.254" layer="121"/>
 <text x="83.82" y="17.399" size="1.778" layer="121" font="vector" ratio="15" rot="R180">IC1</text>
-<text x="78.359" y="22.225" size="1.778" layer="121" font="vector" ratio="15" rot="R90">74154N</text>
+<text x="78.359" y="22.225" size="1.778" layer="121" font="vector" ratio="15" rot="R90">74LS154N</text>
 <wire x1="44.704" y1="36.83" x2="44.704" y2="16.51" width="0.254" layer="121"/>
 <wire x1="50.546" y1="16.51" x2="50.546" y2="36.83" width="0.254" layer="121"/>
@@
 <param name="dpMaxLengthDifference" value="10mm"/>
 <param name="dpGapFactor" value="2.5"/>
-<param name="checkGrid" value="0"/>
-<param name="checkAngle" value="0"/>
+<param name="checkGrid" value="1"/>
+<param name="checkAngle" value="1"/>
 <param name="checkFont" value="1"/>
 <param name="checkRestrict" value="1"/>
@@
 <wire x1="125.73" y1="15.24" x2="121.285" y2="10.795" width="0.8128" layer="1"/>
 <wire x1="140.6525" y1="8.255" x2="136.8425" y2="12.065" width="0.8128" layer="16"/>
-<wire x1="136.8425" y1="12.065" x2="129.54" y2="12.065" width="0.8128" layer="16"/>
-<wire x1="129.54" y1="12.065" x2="125.73" y2="15.24" width="0.8128" layer="16"/>
+<wire x1="136.8425" y1="12.065" x2="128.905" y2="12.065" width="0.8128" layer="16"/>
+<wire x1="128.905" y1="12.065" x2="125.73" y2="15.24" width="0.8128" layer="16"/>
 <wire x1="18.415" y1="16.1925" x2="25.4" y2="16.1925" width="0.8128" layer="1"/>
 <wire x1="25.4" y1="16.1925" x2="26.9875" y2="14.605" width="0.8128" layer="1"/>
@@
 <wire x1="125.73" y1="6.985" x2="125.73" y2="12.065" width="0.4064" layer="16"/>
 <wire x1="125.73" y1="12.065" x2="121.92" y2="15.875" width="0.4064" layer="16"/>
-<wire x1="121.92" y1="15.875" x2="121.92" y2="68.2625" width="0.4064" layer="16"/>
-<wire x1="121.92" y1="68.2625" x2="118.11" y2="71.755" width="0.4064" layer="16"/>
+<wire x1="121.92" y1="15.875" x2="121.92" y2="68.8975" width="0.4064" layer="16"/>
+<wire x1="121.92" y1="68.8975" x2="119.0625" y2="71.755" width="0.4064" layer="16"/>
+<wire x1="119.0625" y1="71.755" x2="118.11" y2="71.755" width="0.4064" layer="16"/>
 </signal>
 <signal name="FZ">
@@
 <wire x1="26.67" y1="69.215" x2="19.05" y2="69.215" width="0.4064" layer="16"/>
 <wire x1="124.46" y1="5.715" x2="123.19" y2="6.985" width="0.4064" layer="16"/>
-<wire x1="120.9675" y1="66.675" x2="118.11" y2="69.215" width="0.4064" layer="16"/>
 <wire x1="123.19" y1="6.985" x2="123.19" y2="13.335" width="0.4064" layer="16"/>
 <wire x1="123.19" y1="13.335" x2="120.9675" y2="15.5575" width="0.4064" layer="16"/>
-<wire x1="120.9675" y1="15.5575" x2="120.9675" y2="66.675" width="0.4064" layer="16"/>
+<wire x1="120.9675" y1="15.5575" x2="120.9675" y2="67.31" width="0.4064" layer="16"/>
+<wire x1="120.9675" y1="67.31" x2="119.0625" y2="69.215" width="0.4064" layer="16"/>
+<wire x1="119.0625" y1="69.215" x2="118.11" y2="69.215" width="0.4064" layer="16"/>
 </signal>
 <signal name="FN">
@@
 <via x="47.3075" y="51.435" extent="1-16" drill="0.6096" diameter="1.27"/>
 <via x="91.44" y="51.435" extent="1-16" drill="0.6096" diameter="1.27"/>
-<wire x1="103.505" y1="16.8275" x2="116.205" y2="16.8275" width="0.4064" layer="16"/>
-<wire x1="116.205" y1="16.8275" x2="116.205" y2="19.685" width="0.4064" layer="1"/>
-<via x="116.205" y="16.8275" extent="1-16" drill="0.6096" diameter="1.27"/>
+<via x="115.57" y="16.51" extent="1-16" drill="0.6096" diameter="1.27"/>
 <wire x1="114.3" y1="21.59" x2="109.855" y2="26.035" width="0.4064" layer="16"/>
 <wire x1="109.855" y1="26.035" x2="109.855" y2="38.1" width="0.4064" layer="16"/>
@@
 <wire x1="94.9325" y1="12.065" x2="98.7425" y2="12.065" width="0.4064" layer="16"/>
 <wire x1="98.7425" y1="12.065" x2="103.505" y2="16.8275" width="0.4064" layer="16"/>
+<wire x1="115.57" y1="16.51" x2="116.205" y2="17.145" width="0.4064" layer="1"/>
+<wire x1="116.205" y1="17.145" x2="116.205" y2="19.685" width="0.4064" layer="1"/>
+<wire x1="103.505" y1="16.8275" x2="115.2525" y2="16.8275" width="0.4064" layer="16"/>
+<wire x1="115.2525" y1="16.8275" x2="115.57" y2="16.51" width="0.4064" layer="16"/>
 </signal>
 <signal name="/MEM2ALULO">
@@
 <via x="41.5925" y="50.165" extent="1-16" drill="0.6096" diameter="1.27"/>
 <via x="90.17" y="50.165" extent="1-16" drill="0.6096" diameter="1.27"/>
-<wire x1="94.615" y1="13.97" x2="95.25" y2="13.97" width="0.4064" layer="16"/>
-<wire x1="95.25" y1="13.97" x2="98.1075" y2="13.97" width="0.4064" layer="16"/>
 <wire x1="98.1075" y1="13.97" x2="104.4575" y2="20.32" width="0.4064" layer="16"/>
-<wire x1="114.3" y1="19.05" x2="108.585" y2="25.0825" width="0.4064" layer="16"/>
 <wire x1="104.4575" y1="20.32" x2="109.855" y2="20.32" width="0.4064" layer="16"/>
 <wire x1="109.855" y1="20.32" x2="111.125" y2="19.05" width="0.4064" layer="16"/>
-<wire x1="111.125" y1="19.05" x2="114.3" y2="19.05" width="0.4064" layer="16"/>
-<wire x1="108.585" y1="25.0825" x2="108.585" y2="36.195" width="0.4064" layer="16"/>
+<wire x1="111.125" y1="19.05" x2="113.665" y2="19.05" width="0.4064" layer="16"/>
+<wire x1="108.585" y1="25.0825" x2="108.585" y2="25.4" width="0.4064" layer="16"/>
 <via x="108.585" y="36.195" extent="1-16" drill="0.6096" diameter="1.27"/>
+<wire x1="108.585" y1="25.4" x2="108.585" y2="36.195" width="0.4064" layer="16"/>
 <wire x1="108.585" y1="36.195" x2="94.615" y2="50.165" width="0.4064" layer="1"/>
 <wire x1="94.615" y1="50.165" x2="90.17" y2="50.165" width="0.4064" layer="1"/>
 <wire x1="88.9" y1="8.255" x2="88.9" y2="12.3825" width="0.4064" layer="16"/>
 <wire x1="88.9" y1="12.3825" x2="90.4875" y2="13.97" width="0.4064" layer="16"/>
-<wire x1="90.4875" y1="13.97" x2="94.615" y2="13.97" width="0.4064" layer="16"/>
+<wire x1="90.4875" y1="13.97" x2="98.1075" y2="13.97" width="0.4064" layer="16"/>
+<wire x1="114.3" y1="19.05" x2="113.665" y2="19.05" width="0.4064" layer="16"/>
+<wire x1="113.665" y1="19.05" x2="108.585" y2="24.13" width="0.4064" layer="16"/>
+<wire x1="108.585" y1="24.13" x2="108.585" y2="25.0825" width="0.4064" layer="16"/>
 </signal>
 <signal name="ALUBUS8">
@@
 <wire x1="98.425" y1="24.13" x2="104.4575" y2="18.0975" width="0.4064" layer="1"/>
 <wire x1="104.4575" y1="18.0975" x2="104.4575" y2="14.2875" width="0.4064" layer="1"/>
-<wire x1="104.4575" y1="14.2875" x2="109.22" y2="9.2075" width="0.4064" layer="16"/>
-<wire x1="109.22" y1="9.2075" x2="109.22" y2="8.255" width="0.4064" layer="16"/>
+<wire x1="109.22" y1="9.525" x2="109.22" y2="8.255" width="0.4064" layer="16"/>
 <via x="104.4575" y="14.2875" extent="1-16" drill="0.6096" diameter="1.27"/>
+<wire x1="109.22" y1="9.525" x2="104.4575" y2="14.2875" width="0.4064" layer="16"/>
 </signal>
 <signal name="/LDMSW">
@@
 <wire x1="39.6875" y1="30.7975" x2="38.735" y2="31.75" width="0.4064" layer="1"/>
 <wire x1="38.735" y1="31.75" x2="32.7025" y2="31.75" width="0.4064" layer="1"/>
-<via x="32.7025" y="31.75" extent="1-16" drill="0.6096"/>
+<via x="32.7025" y="31.75" extent="1-16" drill="0.6096" diameter="1.27"/>
 </signal>
 <signal name="/ENMAR">
@@
 <wire x1="133.35" y1="21.59" x2="132.715" y2="21.59" width="0.4064" layer="16"/>
 <wire x1="132.715" y1="21.59" x2="131.445" y2="22.86" width="0.4064" layer="16"/>
-<wire x1="131.445" y1="22.86" x2="131.445" y2="27.6225" width="0.4064" layer="16"/>
-<wire x1="131.445" y1="27.6225" x2="132.715" y2="29.21" width="0.4064" layer="16"/>
+<wire x1="131.445" y1="22.86" x2="131.445" y2="27.94" width="0.4064" layer="16"/>
+<wire x1="131.445" y1="27.94" x2="132.715" y2="29.21" width="0.4064" layer="16"/>
 <wire x1="132.715" y1="29.21" x2="133.35" y2="29.21" width="0.4064" layer="16"/>
 <wire x1="106.68" y1="8.255" x2="107.95" y2="6.985" width="0.4064" layer="16"/>
@@
 <contactref element="UC4" pad="14"/>
 <contactref element="JP10" pad="11"/>
-<wire x1="114.3" y1="8.255" x2="118.11" y2="59.055" width="0" layer="19" extent="1-1"/>
+<wire x1="114.3" y1="8.255" x2="114.3" y2="9.2075" width="0.4064" layer="16"/>
+<wire x1="114.3" y1="9.2075" x2="117.1575" y2="12.065" width="0.4064" layer="16"/>
+<wire x1="117.1575" y1="12.065" x2="117.1575" y2="42.8625" width="0.4064" layer="16"/>
+<wire x1="117.1575" y1="42.8625" x2="112.7125" y2="47.3075" width="0.4064" layer="16"/>
+<wire x1="112.7125" y1="47.3075" x2="112.7125" y2="59.055" width="0.4064" layer="16"/>
+<wire x1="112.7125" y1="59.055" x2="118.11" y2="59.055" width="0.4064" layer="1"/>
+<via x="112.7125" y="59.055" extent="1-16" drill="0.6096" diameter="1.27"/>
 </signal>
 <signal name="/FRET">
