File: eagle/6_cpu_registers_a.brd (EAGLE design)
At the start: 160 x 100 mm, 39 parts, among them IC1 74LS374N, IC10 74LS374N, IC11 74LS374N, IC12 74LS374N, IC13 74LS374N, IC14 74LS374N, IC2 74LS374N, IC21 74LS08N, IC22 74LS32N, IC3 74LS374N, IC4 74LS374N, IC5 74LS374N, IC6 74LS374N, IC9 74LS374N

Commit message: Sat Feb  6 20:10:54 CET 2016
Other:
- board text added: "#6"
- board text removed: "#5"
Changed lines of the file:
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@@
 <text x="76.581" y="16.8275" size="1.27" layer="121" font="vector" ratio="16" rot="R180">74LS08N</text>
 <text x="100.2665" y="15.875" size="1.27" layer="121" font="vector" ratio="16">74LS32N</text>
-<text x="147.0025" y="86.6775" size="3.81" layer="1" font="vector" ratio="15">#5</text>
+<text x="147.0025" y="86.6775" size="3.81" layer="1" font="vector" ratio="15">#6</text>
 </plain>
 <attributes>

Commit message: 2016-02-10 17:30 (completed boards 2,6,7)
Parts:
- JP10: device pinhead:2X16 -> pinhead:2X18
- moved JP10 2.54 mm to (105.4, 6.99)
- moved C2 0.63 mm to (80.0, 9.84)
Connections:
- new net /FP: JP10.34
- new net /IO: JP10.35
- new net /MEMOP: JP10.11
- new net /NP_FAULT: JP10.36
- new net /WR_FAULT: JP10.33
Routing:
- net +5V: track 526.0 -> 528.0 mm
- net MDRLDINHBT: track 98.8 -> 100.3 mm
