File: eagle/6_cpu_registers_a.sch (EAGLE design)
At the start: 39 parts, among them IC1 74LS374N, IC10 74LS374N, IC11 74LS374N, IC12 74LS374N, IC13 74LS374N, IC14 74LS374N, IC2 74LS374N, IC21 74LS08N, IC22 74LS32N, IC3 74LS374N, IC4 74LS374N, IC5 74LS374N, IC6 74LS374N, IC9 74LS374N

Commit message: 2016-02-10 17:30 (completed boards 2,6,7)
Parts:
- JP10: device pinhead:PINHD-2X16 -> pinhead:PINHD-2X18
Connections:
- new net /FP: JP10.34
- new net /IO: JP10.35
- new net /MEMOP: JP10.11
- new net /NP_FAULT: JP10.36
- new net /WR_FAULT: JP10.33
Changed lines of the file:
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@@
 <part name="JP3" library="pinhead" deviceset="PINHD-2X8" device=""/>
 <part name="JP4" library="pinhead" deviceset="PINHD-2X8" device=""/>
-<part name="JP10" library="pinhead" deviceset="PINHD-2X16" device=""/>
+<part name="JP10" library="pinhead" deviceset="PINHD-2X18" device=""/>
 <part name="JP9" library="pinhead" deviceset="PINHD-2X24" device=""/>
 <part name="JP5" library="pinhead" deviceset="PINHD-2X8" device=""/>
@@
 <instance part="JP3" gate="A" x="154.94" y="226.06"/>
 <instance part="JP4" gate="A" x="154.94" y="187.96"/>
-<instance part="JP10" gate="A" x="86.36" y="134.62"/>
+<instance part="JP10" gate="A" x="86.36" y="132.08"/>
 <instance part="JP9" gate="A" x="86.36" y="68.58"/>
 <instance part="JP5" gate="A" x="213.36" y="187.96"/>
@@
 </segment>
 </net>
+<net name="/MEMOP" class="0">
+<segment>
+<pinref part="JP10" gate="A" pin="11"/>
+<wire x1="83.82" y1="139.7" x2="73.66" y2="139.7" width="0.1524" layer="91"/>
+<label x="73.66" y="139.7" size="1.27" layer="95" rot="R180" xref="yes"/>
+</segment>
+</net>
+<net name="/WR_FAULT" class="0">
+<segment>
+<pinref part="JP10" gate="A" pin="33"/>
+<wire x1="83.82" y1="111.76" x2="73.66" y2="111.76" width="0.1524" layer="91"/>
+<label x="73.66" y="111.76" size="1.27" layer="95" rot="R180" xref="yes"/>
+</segment>
+</net>
+<net name="/IO" class="0">
+<segment>
+<pinref part="JP10" gate="A" pin="35"/>
+<wire x1="83.82" y1="109.22" x2="73.66" y2="109.22" width="0.1524" layer="91"/>
+<label x="73.66" y="109.22" size="1.27" layer="95" rot="R180" xref="yes"/>
+</segment>
+</net>
+<net name="/FP" class="0">
+<segment>
+<pinref part="JP10" gate="A" pin="34"/>
+<wire x1="91.44" y1="111.76" x2="101.6" y2="111.76" width="0.1524" layer="91"/>
+<label x="101.6" y="111.76" size="1.27" layer="95" xref="yes"/>
+</segment>
+</net>
+<net name="/NP_FAULT" class="0">
+<segment>
+<pinref part="JP10" gate="A" pin="36"/>
+<wire x1="91.44" y1="109.22" x2="101.6" y2="109.22" width="0.1524" layer="91"/>
+<label x="101.6" y="109.22" size="1.27" layer="95" xref="yes"/>
+</segment>
+</net>
