File: eagle/7_cpu_registers_b.brd (EAGLE design)
At the start: 160 x 100 mm, 47 parts, among them IC1 74LS569, IC10 74LS157N, IC11 74LS157N, IC12 74LS569, IC13 74LS569, IC14 74LS569, IC15 74LS569, IC16 74LS569, IC17 74LS569, IC18 74LS569, IC19 74LS569, IC2 74LS569, IC3 74LS569, IC4 74LS569, IC5 74LS569, IC6 74LS569, IC7 74LS569, IC8 74LS569, IC9 74LS08N

Commit message: Sat Feb  6 20:10:54 CET 2016
Other:
- board text added: "#7"
- board text removed: "#6"
Changed lines of the file:
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@@
 <text x="55.626" y="54.229" size="1.27" layer="121" font="vector" ratio="16">74LS569</text>
 <text x="24.8285" y="54.229" size="1.27" layer="121" font="vector" ratio="16">74LS569</text>
-<text x="7.3025" y="22.5425" size="3.81" layer="1" font="vector" ratio="15">#6</text>
+<text x="7.3025" y="22.5425" size="3.81" layer="1" font="vector" ratio="15">#7</text>
 <circle x="165.1" y="-4.7625" radius="2.159" width="0.2032" layer="100"/>
 <wire x1="165.1" y1="0" x2="165.1" y2="-9.525" width="0.2032" layer="100"/>

Commit message: 2016-02-10 17:30 (completed boards 2,6,7)
Parts:
- JP10: device pinhead:2X16 -> pinhead:2X18
- moved JP10 2.54 mm to (105.4, 6.99)
Connections:
- new net /FP: JP10.34
- new net /IO: JP10.35
- new net /MEMOP: JP10.11
- new net /NP_FAULT: JP10.36
- new net /WR_FAULT: JP10.33
Routing:
- net /LDSP: track 187.5 -> 189.0 mm
