File: eagle/7_cpu_registers_b.sch (EAGLE design)
At the start: 47 parts, among them IC1 74LS569, IC10 74LS157N, IC11 74LS157N, IC12 74LS569, IC13 74LS569, IC14 74LS569, IC15 74LS569, IC16 74LS569, IC17 74LS569, IC18 74LS569, IC19 74LS569, IC2 74LS569, IC3 74LS569, IC4 74LS569, IC5 74LS569, IC6 74LS569, IC7 74LS569, IC8 74LS569, IC9 74LS08N

Commit message: Sat Feb  6 20:10:54 CET 2016
Other:
- note added: "CPU.7"
- note removed: "CPU.5"
Changed lines of the file:
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@@
 <text x="386.08" y="33.02" size="2.54" layer="97" font="vector" rot="R180">Dawid Pilawa</text>
 <text x="386.08" y="27.94" size="2.54" layer="97" font="vector" rot="R180">(C) 2010-2014</text>
-<text x="370.84" y="10.16" size="2.54" layer="97" font="vector" rot="R180">CPU.5</text>
+<text x="370.84" y="10.16" size="2.54" layer="97" font="vector" rot="R180">CPU.7</text>
 <text x="386.08" y="10.16" size="2.54" layer="97" font="vector" rot="R180">1.5</text>
 </plain>
@@
 <text x="386.08" y="33.02" size="2.54" layer="97" font="vector" rot="R180">Dawid Pilawa</text>
 <text x="386.08" y="27.94" size="2.54" layer="97" font="vector" rot="R180">(C) 2010-2014</text>
-<text x="370.84" y="10.16" size="2.54" layer="97" font="vector" rot="R180">CPU.5</text>
+<text x="370.84" y="10.16" size="2.54" layer="97" font="vector" rot="R180">CPU.7</text>
 <text x="386.08" y="10.16" size="2.54" layer="97" font="vector" rot="R180">1.5</text>
 <text x="10.16" y="246.38" size="6.4516" layer="91">BOARD CONNECTORS</text>

Commit message: 2016-02-10 17:30 (completed boards 2,6,7)
Parts:
- JP10: device pinhead:PINHD-2X16 -> pinhead:PINHD-2X18
Connections:
- new net /FP: JP10.34
- new net /IO: JP10.35
- new net /MEMOP: JP10.11
- new net /NP_FAULT: JP10.36
- new net /WR_FAULT: JP10.33
Other:
- note added: "(C) 2010-2016"
- note added: "2.0"
- note removed: "(C) 2010-2014"
- note removed: "1.5"
Changed lines of the file:
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@@
 <part name="SUPPLY34" library="supply2" deviceset="GND" device=""/>
 <part name="JP3" library="pinhead" deviceset="PINHD-2X8" device=""/>
-<part name="JP10" library="pinhead" deviceset="PINHD-2X16" device=""/>
+<part name="JP10" library="pinhead" deviceset="PINHD-2X18" device=""/>
 <part name="JP9" library="pinhead" deviceset="PINHD-2X24" device=""/>
 <part name="FRAME2" library="frames" deviceset="DINA3_L" device=""/>
@@
 <text x="289.56" y="27.94" size="2.54" layer="97" font="vector">Registers (MAR,PC,KSP,SP)</text>
 <text x="386.08" y="33.02" size="2.54" layer="97" font="vector" rot="R180">Dawid Pilawa</text>
-<text x="386.08" y="27.94" size="2.54" layer="97" font="vector" rot="R180">(C) 2010-2014</text>
+<text x="386.08" y="27.94" size="2.54" layer="97" font="vector" rot="R180">(C) 2010-2016</text>
 <text x="370.84" y="10.16" size="2.54" layer="97" font="vector" rot="R180">CPU.7</text>
-<text x="386.08" y="10.16" size="2.54" layer="97" font="vector" rot="R180">1.5</text>
+<text x="386.08" y="10.16" size="2.54" layer="97" font="vector" rot="R180">2.0</text>
 </plain>
 <instances>
@@
 <text x="289.56" y="27.94" size="2.54" layer="97" font="vector">Registers (MAR,PC,KSP,SP)</text>
 <text x="386.08" y="33.02" size="2.54" layer="97" font="vector" rot="R180">Dawid Pilawa</text>
-<text x="386.08" y="27.94" size="2.54" layer="97" font="vector" rot="R180">(C) 2010-2014</text>
+<text x="386.08" y="27.94" size="2.54" layer="97" font="vector" rot="R180">(C) 2010-2016</text>
 <text x="370.84" y="10.16" size="2.54" layer="97" font="vector" rot="R180">CPU.7</text>
-<text x="386.08" y="10.16" size="2.54" layer="97" font="vector" rot="R180">1.5</text>
+<text x="386.08" y="10.16" size="2.54" layer="97" font="vector" rot="R180">2.0</text>
 <text x="10.16" y="246.38" size="6.4516" layer="91">BOARD CONNECTORS</text>
 </plain>
@@
 <instance part="SUPPLY34" gate="GND" x="33.02" y="175.26"/>
 <instance part="JP3" gate="A" x="154.94" y="226.06"/>
-<instance part="JP10" gate="A" x="86.36" y="134.62"/>
+<instance part="JP10" gate="A" x="86.36" y="132.08"/>
 <instance part="JP9" gate="A" x="86.36" y="68.58"/>
 </instances>
@@
 </segment>
 </net>
+<net name="/MEMOP" class="0">
+<segment>
+<pinref part="JP10" gate="A" pin="11"/>
+<wire x1="83.82" y1="139.7" x2="73.66" y2="139.7" width="0.1524" layer="91"/>
+<label x="73.66" y="139.7" size="1.27" layer="95" rot="R180" xref="yes"/>
+</segment>
+</net>
+<net name="/WR_FAULT" class="0">
+<segment>
+<pinref part="JP10" gate="A" pin="33"/>
+<wire x1="83.82" y1="111.76" x2="73.66" y2="111.76" width="0.1524" layer="91"/>
+<label x="73.66" y="111.76" size="1.27" layer="95" rot="R180" xref="yes"/>
+</segment>
+</net>
+<net name="/IO" class="0">
+<segment>
+<pinref part="JP10" gate="A" pin="35"/>
+<wire x1="83.82" y1="109.22" x2="73.66" y2="109.22" width="0.1524" layer="91"/>
+<label x="73.66" y="109.22" size="1.27" layer="95" rot="R180" xref="yes"/>
+</segment>
+</net>
+<net name="/NP_FAULT" class="0">
+<segment>
+<pinref part="JP10" gate="A" pin="36"/>
+<wire x1="91.44" y1="109.22" x2="101.6" y2="109.22" width="0.1524" layer="91"/>
+<label x="101.6" y="109.22" size="1.27" layer="95" xref="yes"/>
+</segment>
+</net>
+<net name="/FP" class="0">
+<segment>
+<pinref part="JP10" gate="A" pin="34"/>
+<wire x1="91.44" y1="111.76" x2="101.6" y2="111.76" width="0.1524" layer="91"/>
+<label x="101.6" y="111.76" size="1.27" layer="95" xref="yes"/>
+</segment>
+</net>
