File: eagle/4_cpu_control.brd (EAGLE design)
At the start: 160 x 100 mm, 50 parts, among them IC1 74LS151N, IC10 74LS173N, IC11 74LS74N, IC12 74LS74N, IC13 74LS541N, IC14 74LS541N, IC15 74LS21N, IC16 74LS02N, IC17 74LS02N, IC18 74LS04N, IC2 74LS151N, IC20 74LS08N, IC3 74LS153N, IC4 74LS153N, IC5 74LS541N, IC6 74LS32N, IC7 74LS08N, IC8 74LS151N, IC9 74LS157N

Commit message: Sat Feb  6 20:10:54 CET 2016
Other:
- board text added: "#4"
- board text removed: "#3"
Changed lines of the file:
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@@
 <circle x="157.1625" y="94.615" radius="2.286" width="0" layer="43"/>
 <circle x="3.4925" y="5.715" radius="2.286" width="0" layer="43"/>
-<text x="143.8275" y="80.9625" size="3.81" layer="1" font="vector" ratio="15">#3</text>
+<text x="143.8275" y="80.9625" size="3.81" layer="1" font="vector" ratio="15">#4</text>
 <circle x="-4.7625" y="104.775" radius="2.159" width="0.2032" layer="100"/>
 <wire x1="-4.7625" y1="100.0125" x2="-4.7625" y2="109.5375" width="0.2032" layer="100"/>

Commit message: 2016-02-10 17:30 (completed boards 2,6,7)
Connections:
- removed net /ENPPC: JP9.37
Changed lines of the file:
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@@
 <contactref element="JP9" pad="41"/>
-</signal>
-<signal name="/ENPPC">
-<contactref element="JP9" pad="37"/>
 </signal>
 <signal name="/ENMAR">

Commit message: Wed Feb 10 22:17:37 CET 2016 (completed boards 5,4)
Connections:
- new net /MEMOP: JP10.11
