File: eagle/4_cpu_control.sch (EAGLE design)
At the start: 41 parts, among them IC1 74LS08N, IC10 74LS173N, IC11 74LS273N, IC12 74LS74N, IC13 74LS157N, IC14 74LS157N, IC2 74LS163, IC3 74LS163, IC4 74LS00N, IC5 74LS273N, IC6 74LS148N, IC7 74LS148N, IC8 74LS08N, IC9 74S32N

Commit message: Renumbered boards and schematic sheets
Parts:
- removed JP1: (no value), pinhead:PINHD-2X8
- removed JP8: (no value), pinhead:PINHD-1X5
- removed RN1: 4.7k, resistor-sil:G08R
- added C16, C17, C18, C19: 100n, rcl:C-EU050-024X044
- added C20: 10u, rcl:CPOL-EUE2.5-6
- added IC15: 74LS21N, 74xx-eu:74LS21N
- added IC16, IC17: 74LS02N, 74xx-eu:74LS02N
- added IC18: 74LS04N, 74xx-eu:74LS04N
- added IC20: 74LS08N, 74xx-eu:74LS08N
- added JP5: (no value), pinhead:PINHD-2X8
- added JP9: (no value), pinhead:PINHD-2X24
- C15: value 10u -> 100n; device rcl:CPOL-EUE5-6 -> rcl:C-EU050-024X044
- IC1, IC8: value 74LS08N -> 74LS151N; device 74xx-eu:74LS08N -> 74xx-eu:74LS151N
- IC11: value 74LS273N -> 74LS74N; device 74xx-eu:74273N -> 74xx-eu:74LS74N
- IC13, IC14: value 74LS157N -> 74LS541N; device 74xx-eu:74LS157N -> 74xx-us:74LS541N
- IC2: value 74LS163 -> 74LS151N; device 74xx-eu:74160N -> 74xx-eu:74LS151N
- IC3: value 74LS163 -> 74LS153N; device 74xx-eu:74160N -> 74xx-eu:74LS153N
- IC4: value 74LS00N -> 74LS153N; device 74xx-eu:74LS00N -> 74xx-eu:74LS153N
- IC5: value 74LS273N -> 74LS541N; device 74xx-eu:74273N -> 74xx-us:74LS541N
- IC6: value 74LS148N -> 74LS32N; device 74xx-eu:74LS148N -> 74xx-eu:74LS32N
- IC7: value 74LS148N -> 74LS08N; device 74xx-eu:74LS148N -> 74xx-eu:74LS08N
- IC9: value 74S32N -> 74LS157N; device 74xx-eu:74S32N -> 74xx-eu:74LS157N
Connections:
- removed net /FAULT_PF: IC4C.O, IC7A.7
- removed net /NEXTOP: IC10A.G1, IC10A.G2, IC1B.O, IC9D.I0
- removed net CNT0: IC2A.QA, JP8.1
- removed net CNT1: IC2A.QB, JP8.2
- removed net CNT2: IC2A.QC, JP8.3
- removed net CNT3: IC2A.QD, JP8.4
- removed net CNT4: IC3A.QA, JP8.5
- removed net DBUS0: IC11A.D1, JP1.1
- removed net DBUS1: IC11A.D2, JP1.3
- removed net DBUS2: IC11A.D3, JP1.5
- removed net DBUS3: IC11A.D4, JP1.7
- removed net DBUS4: IC11A.D5, JP1.9
- removed net DBUS5: IC11A.D6, JP1.11
- removed net DBUS6: IC11A.D7, JP1.13
- removed net DBUS7: IC11A.D8, JP1.15
- removed net IRQ0: IC5A.D8, JP1.2, RN1.9
- removed net IRQ1: IC5A.D7, JP1.4, RN1.8
- removed net IRQ2: IC5A.D6, JP1.6, RN1.7
- removed net IRQ3: IC5A.D5, JP1.8, RN1.6
- removed net IRQ4: IC5A.D4, JP1.10, RN1.5
- removed net IRQ5: IC5A.D3, JP1.12, RN1.4
- removed net IRQ6: IC5A.D2, JP1.14, RN1.3
- removed net IRQ7: IC5A.D1, JP1.16, RN1.2
- removed net N$18: IC10A.Q1, IC13A.1A
- removed net N$20: IC10A.Q3, IC13A.3A
- removed net N$22: IC11A.Q8, IC14A.4B
- removed net N$23: IC11A.Q7, IC14A.3B
- removed net N$24: IC11A.Q6, IC14A.2B
- removed net N$25: IC11A.Q5, IC14A.1B
- removed net N$26: IC11A.Q1, IC13A.1B
- removed net N$27: IC6A.EI, IC9B.O
- removed net N$28: IC11A.Q3, IC13A.3B
- removed net N$30: IC11A.Q4, IC13A.4B
- removed net N$4: IC6A.A1, IC8B.I0
- removed net N$47: IC12A.Q, IC13A.!A!/B, IC14A.!A!/B
- removed net N$5: IC7A.A1, IC8B.I1
- removed net N$57: IC5A.Q8, IC6A.7
- removed net N$58: IC5A.Q7, IC6A.6
- removed net N$59: IC5A.Q6, IC6A.5
- removed net N$60: IC5A.Q5, IC6A.4
- removed net N$61: IC5A.Q4, IC6A.3
- removed net N$62: IC5A.Q3, IC6A.2
- removed net N$63: IC5A.Q2, IC6A.1
- removed net N$64: IC5A.Q1, IC6A.0
- new net /ALUCARRYIN: JP9.2
- new net /ALUSHR: IC1A.C, JP9.1
- new net /CARRY1: IC18B.I, JP9.29
- new net /CARRY3: IC18A.I, JP9.31
- new net /ENA: JP9.33
- new net /ENALU: JP9.39
- new net /ENDP: JP9.44
- new net /ENIPTR: IC13A.G1, IC13A.G2, IC14A.G1, IC14A.G2, JP9.38
- new net /ENLMDR: JP9.34
- new net /ENMAR: JP9.48
- new net /ENMSW: IC5A.G1, IC5A.G2, JP9.40
- new net /ENPC: JP9.42
- new net /ENPPC: JP9.37
- new net /ENRMDR: JP9.41
- new net /ENSP: JP9.46
- new net /ENX: JP9.36
- new net /ENY: JP9.35
- new net /INC_MAR: JP9.32
- new net /LATCH_I: IC7B.I1, JP9.47
- new net /LATCH_S: IC7C.I1, JP9.45
- new net /LDA: JP9.14
- new net /LDAHI: JP9.11
- new net /LDALO: JP9.12
- new net /LDDP: JP9.22
- new net /LDMAR: JP9.23
- new net /LDMARHI: JP9.17
- new net /LDMARLO: JP9.18
- new net /LDMDR: JP9.9
- new net /LDMDRHI: JP9.10
- new net /LDMDRLO: JP9.7
- new net /LDMSW: IC11A.CLK, IC11B.CLK, IC7B.I0, IC7C.I0, IC7D.I1, IC9A.!A!/B, JP9.20
- new net /LDPC: JP9.19
- new net /LDSP: JP9.21
- new net /LDX: JP9.13
- new net /LDY: JP9.16
- new net ALUMODE: JP9.3
- new net ALUOP0: JP9.4
- new net ALUOP1: IC18D.I, IC2A.D3, IC2A.D4, IC8A.D3, IC8A.D4, JP9.6
- new net ALUOP2: JP9.5
- new net ALUOP3: JP9.8
- new net ALURES0: IC1A.D0, IC1A.D2, JP9.25
- new net ALURES8: IC1A.D1, JP9.27
- new net ALU_C: IC1A.Y, IC9A.1B
- new net ALU_N: IC3A.1Y, IC9A.3B
- new net ALU_V: IC4A.1Y, IC9A.4B
- new net ALU_Z: IC3A.2Y, IC9A.2B
- new net F7: IC11A.Q, IC5A.A8
- new net LBUS0: JP5.15
- new net LBUS1: JP5.16
- new net LBUS10: JP5.5
- new net LBUS11: JP5.6
- new net LBUS12: JP5.3
- new net LBUS13: JP5.4
- new net LBUS14: JP5.1
- new net LBUS15: IC8A.C, JP5.2
- new net LBUS2: JP5.13
- new net LBUS3: JP5.14
- new net LBUS4: JP5.11
- new net LBUS5: JP5.12
- new net LBUS6: JP5.9
- new net LBUS7: IC2A.C, JP5.10
- new net LBUS8: JP5.7
- new net LBUS9: JP5.8
- new net LOAD_FLAGS0: IC1A.A, IC3A.A, IC4A.A, IC7A.I0, JP9.24
- new net LOAD_FLAGS1: IC1A.B, IC3A.B, IC4A.B, IC7A.I1, JP9.26
- new net MDRLDINHBT: JP9.43
- new net N$32: IC10A.D1, IC9A.1Y
- new net N$48: IC10A.D2, IC9A.2Y
- new net N$49: IC10A.D3, IC9A.3Y
- new net N$50: IC10A.D4, IC9A.4Y
- new net N$51: IC7A.O, IC7D.I0
- new net N$52: IC12A.CLK, IC6C.O
- new net N$53: IC12B.CLK, IC6D.O
- new net N$54: IC6C.I1, IC7B.O
- new net N$55: IC6D.I1, IC7C.O
- net +5V: now also C15.1, C16.1, C17.1, C18.1, C19.1, C20.+, IC11A.CLR, IC11A.PRE, IC11B.CLR, IC12B.PRE, IC15P.VCC, IC16P.VCC, IC17P.VCC, IC18C.I, IC18E.I, IC18F.I, IC18P.VCC, IC20B.I0, IC20B.I1, IC20C.I0, IC20C.I1, IC20D.I0, IC20D.I1, IC20P.VCC, IC4A.2C0, IC4A.2C1, IC4A.2C2, IC4A.2C3, IC4A.2G, IC6A.I0, IC6A.I1, IC6B.I0, IC6B.I1; no longer C15.+, IC1C.I0, IC1C.I1, IC1D.I0, IC1D.I1, IC2A.ENP, IC2A.ENT, IC2A.LD, IC3A.LD, IC4A.I0, IC4A.I1, IC4B.I0, IC4B.I1, IC5A.CLR, IC7A.0, IC7A.1, IC7A.2, IC7A.3, IC7A.4, IC9A.I0, IC9A.I1, IC9C.I0, IC9C.I1, RN1.1
- net /BUSIFCEN: no longer IC4D.I1
- net /FI: now also IC12A.Q, IC5A.A5; no longer IC9B.I0
- net /FP: now also IC11B.Q, IC5A.A7
- net /FS: now also IC12B.Q, IC5A.A6; no longer IC4C.I0
- net /LATCHFLAGS: no longer IC4D.O
- net /LOAD_IR: no longer IC1A.I1
- net /NP_FAULT: no longer IC7A.6
- net /RST: now also IC11B.PRE, IC12B.CLR; no longer IC11A.CLR, IC1A.I0
- net /WR_FAULT: no longer IC7A.5
- net ALUBUS0: now also IC17A.I0, IC9A.1A
- net ALUBUS1: now also IC17A.I1, IC9A.2A
- net ALUBUS10: now also IC16B.I0
- net ALUBUS11: now also IC16B.I1
- net ALUBUS12: now also IC16C.I0
- net ALUBUS13: now also IC16C.I1
- net ALUBUS14: now also IC16D.I0
- net ALUBUS15: now also IC16D.I1, IC3A.1C0, IC3A.1C1, IC8A.A
- net ALUBUS2: now also IC17B.I0, IC9A.3A
- net ALUBUS3: now also IC17B.I1, IC9A.4A
- net ALUBUS4: now also IC12A.D, IC17C.I0
- net ALUBUS5: now also IC12B.D, IC17C.I1
- net ALUBUS6: now also IC11B.D, IC17D.I0
- net ALUBUS7: now also IC11A.D, IC17D.I1, IC2A.A, IC3A.1C2
- net ALUBUS8: now also IC16A.I0
- net ALUBUS9: now also IC16A.I1
- net BUSCLKA: no longer IC9D.I1
- net BUSCLKB: now also IC6C.I0, IC6D.I0
- net CLK0A: no longer IC10A.CLK, IC2A.CLK, IC3A.CLK, IC5A.CLK
- net CLK0D: now also IC10A.CLK
- net FAULT: no longer IC7A.EO, IC9B.I1
- net FC: now also IC10A.Q1, IC5A.A1
- net FN: now also IC10A.Q3, IC5A.A3
- net FV: now also IC10A.Q4, IC5A.A4
- net FZ: now also IC10A.Q2, IC5A.A2
- net GND: now also C15.2, C16.2, C17.2, C18.2, C19.2, C20.-, IC13A.A1, IC13A.A6, IC13A.A7, IC13A.A8, IC14A.A1, IC14A.A2, IC14A.A3, IC14A.A4, IC14A.A5, IC14A.A6, IC14A.A7, IC14A.A8, IC15P.GND, IC16P.GND, IC17P.GND, IC18P.GND, IC1A.D3, IC1A.D7, IC1A.G, IC20P.GND, IC2A.D0, IC2A.D2, IC2A.D5, IC2A.D7, IC2A.G, IC3A.1C3, IC3A.1G, IC3A.2C3, IC3A.2G, IC4A.1C3, IC4A.1G, IC8A.D0, IC8A.D2, IC8A.D5, IC8A.D7, IC8A.G, IC9A.G; no longer C15.-, IC12B.CLK, IC12B.CLR, IC12B.D, IC12B.PRE, IC13A.G, IC14A.1A, IC14A.2A, IC14A.3A, IC14A.4A, IC14A.G, IC2A.A, IC2A.B, IC2A.C, IC2A.D, IC3A.A, IC3A.B, IC3A.C, IC3A.D, IC7A.EI
- net N$1: now also IC4A.1C0, IC4A.1C1, IC8A.Y; no longer IC6A.A0, IC8A.I0
- net N$10: now also IC15B.I0, IC17A.O; no longer IC1B.I1, IC4D.I0, IC7A.GS, IC8D.I1
- net N$11: now also IC15B.I1, IC17B.O; no longer IC10A.D1, IC8A.O
- net N$12: now also IC15B.I2, IC17C.O; no longer IC10A.D2, IC8B.O
- net N$13: now also IC15B.I3, IC17D.O; no longer IC10A.D3, IC8C.O
- net N$14: now also IC15A.O, IC20A.I0, IC3A.2C1; no longer IC12A.D, IC8D.O
- net N$15: now also IC15B.O, IC20A.I1, IC3A.2C2; no longer IC1A.O, IC1B.I0
- net N$16: now also IC20A.O, IC3A.2C0; no longer IC11A.Q2, IC13A.2B
- net N$17: now also IC10A.G1, IC10A.G2, IC7D.O; no longer IC11A.CLK, IC12A.CLK, IC9D.O
- net N$19: now also IC2A.Y, IC4A.1C2; no longer IC10A.Q2, IC13A.2A
- net N$2: now also IC18B.O, IC1A.D6; no longer IC2A.RCO, IC3A.ENP, IC3A.ENT
- net N$21: now also IC18D.O, IC2A.D1, IC2A.D6, IC8A.D1, IC8A.D6; no longer IC10A.Q4, IC13A.4A
- net N$3: now also IC18A.O, IC1A.D4, IC1A.D5; no longer IC7A.A0, IC8A.I1
- net N$6: now also IC15A.I0, IC16A.O; no longer IC7A.A2, IC8C.I1
- net N$7: now also IC15A.I1, IC16B.O; no longer IC6A.A2, IC8C.I0
- net N$8: now also IC15A.I2, IC16C.O; no longer IC2A.CLR, IC3A.CLR
- net N$9: now also IC15A.I3, IC16D.O; no longer IC10A.D4, IC6A.GS, IC8D.I0
- net OP0: now also IC13A.A2; no longer IC13A.1Y
- net OP1: now also IC13A.A3; no longer IC13A.2Y
- net OP2: now also IC13A.A4; no longer IC13A.3Y
- net OP3: now also IC13A.A5; no longer IC13A.4Y
- net OP4: no longer IC14A.1Y
- net OP5: no longer IC14A.2Y
- net OP6: no longer IC14A.3Y
- net OP7: no longer IC14A.4Y
- net OP8: no longer IC12A.!Q
- net PROT: no longer IC4C.I1
- net RBUS0: now also IC13A.Y1, IC5A.Y1
- net RBUS1: now also IC13A.Y2, IC5A.Y2
- net RBUS10: now also IC14A.Y3
- net RBUS11: now also IC14A.Y4
- net RBUS12: now also IC14A.Y5
- net RBUS13: now also IC14A.Y6
- net RBUS14: now also IC14A.Y7
- net RBUS15: now also IC14A.Y8, IC8A.B
- net RBUS2: now also IC13A.Y3, IC5A.Y3
- net RBUS3: now also IC13A.Y4, IC5A.Y4
- net RBUS4: now also IC13A.Y5, IC5A.Y5
- net RBUS5: now also IC13A.Y6, IC5A.Y6
- net RBUS6: now also IC13A.Y7, IC5A.Y7
- net RBUS7: now also IC13A.Y8, IC2A.B, IC5A.Y8
- net RBUS8: now also IC14A.Y1
- net RBUS9: now also IC14A.Y2
Other:
- note added: "CPU.3"
- note added: "Control (MSW, ALU flags)"
- note removed: "CPU.1"
- note removed: "Control (ucode sequencer)"
- moved on the sheet: C1, C10, C11, C12, C13, C14, C2, C3, C4, C5, C6, C7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

Commit message: Sat Feb  6 20:10:54 CET 2016
Other:
- note added: "CPU.4"
- note removed: "CPU.3"
Changed lines of the file:
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@@
 <text x="208.28" y="-106.68" size="2.54" layer="97" font="vector" rot="R180">Dawid Pilawa</text>
 <text x="208.28" y="-111.76" size="2.54" layer="97" font="vector" rot="R180">(C) 2010-2014</text>
-<text x="193.04" y="-129.54" size="2.54" layer="97" font="vector" rot="R180">CPU.3</text>
+<text x="193.04" y="-129.54" size="2.54" layer="97" font="vector" rot="R180">CPU.4</text>
 </plain>
 <instances>
@@
 <text x="386.08" y="33.02" size="2.54" layer="97" font="vector" rot="R180">Dawid Pilawa</text>
 <text x="386.08" y="27.94" size="2.54" layer="97" font="vector" rot="R180">(C) 2010-2014</text>
-<text x="370.84" y="10.16" size="2.54" layer="97" font="vector" rot="R180">CPU.3</text>
+<text x="370.84" y="10.16" size="2.54" layer="97" font="vector" rot="R180">CPU.4</text>
 <text x="10.16" y="246.38" size="6.4516" layer="91">BOARD CONNECTORS</text>
 </plain>

Commit message: 2016-02-10 17:30 (completed boards 2,6,7)
Connections:
- removed net /ENPPC: JP9.37
Changed lines of the file:
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@@
-</segment>
-</net>
-<net name="/ENPPC" class="0">
-<segment>
-<wire x1="83.82" y1="50.8" x2="73.66" y2="50.8" width="0.1524" layer="91"/>
-<pinref part="JP9" gate="A" pin="37"/>
-<label x="73.66" y="50.8" size="1.27" layer="95" rot="R180" xref="yes"/>
 </segment>
 </net>

Commit message: Wed Feb 10 22:17:37 CET 2016 (completed boards 5,4)
Connections:
- new net /MEMOP: JP10.11
Other:
- note added: "(C) 2010-2016"
- note removed: "(C) 2010-2014"
Changed lines of the file:
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@@
 <text x="208.28" y="-129.54" size="2.54" layer="97" font="vector" rot="R180">2.0</text>
 <text x="208.28" y="-106.68" size="2.54" layer="97" font="vector" rot="R180">Dawid Pilawa</text>
-<text x="208.28" y="-111.76" size="2.54" layer="97" font="vector" rot="R180">(C) 2010-2014</text>
+<text x="208.28" y="-111.76" size="2.54" layer="97" font="vector" rot="R180">(C) 2010-2016</text>
 <text x="193.04" y="-129.54" size="2.54" layer="97" font="vector" rot="R180">CPU.4</text>
 </plain>
@@
 <text x="386.08" y="10.16" size="2.54" layer="97" font="vector" rot="R180">2.0</text>
 <text x="386.08" y="33.02" size="2.54" layer="97" font="vector" rot="R180">Dawid Pilawa</text>
-<text x="386.08" y="27.94" size="2.54" layer="97" font="vector" rot="R180">(C) 2010-2014</text>
+<text x="386.08" y="27.94" size="2.54" layer="97" font="vector" rot="R180">(C) 2010-2016</text>
 <text x="370.84" y="10.16" size="2.54" layer="97" font="vector" rot="R180">CPU.4</text>
 <text x="10.16" y="246.38" size="6.4516" layer="91">BOARD CONNECTORS</text>
@@
 </segment>
 </net>
+<net name="/MEMOP" class="0">
+<segment>
+<pinref part="JP10" gate="A" pin="11"/>
+<wire x1="83.82" y1="139.7" x2="73.66" y2="139.7" width="0.1524" layer="91"/>
+<label x="73.66" y="139.7" size="1.27" layer="95" rot="R180" xref="yes"/>
+</segment>
+</net>
