File: eagle/5_cpu_alu.brd (EAGLE design)
At the start: 160 x 100 mm, 33 parts, among them IC1 74LS181N, IC11 74LS244N, IC12 74LS244N, IC13 74LS244N, IC14 74LS244N, IC18 74LS04N, IC19 74LS32N, IC2 74LS181N, IC3 74LS181N, IC4 74LS181N, IC5 74S182N

Commit message: Sat Feb  6 20:10:54 CET 2016
Other:
- board text added: "#5"
- board text removed: "#4"
Changed lines of the file:
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@@
 <wire x1="-4.7625" y1="100.0125" x2="-4.7625" y2="109.5375" width="0.2032" layer="100"/>
 <wire x1="0" y1="104.775" x2="-9.525" y2="104.775" width="0.2032" layer="100"/>
-<text x="126.6825" y="91.7575" size="3.81" layer="1" font="vector" ratio="15">#4</text>
+<text x="126.6825" y="91.7575" size="3.81" layer="1" font="vector" ratio="15">#5</text>
 </plain>
 <attributes>

Commit message: 2016-02-09 18:12
Changed lines of the file:
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@@
 <param name="dpMaxLengthDifference" value="10mm"/>
 <param name="dpGapFactor" value="2.5"/>
-<param name="checkGrid" value="0"/>
-<param name="checkAngle" value="0"/>
+<param name="checkGrid" value="1"/>
+<param name="checkAngle" value="1"/>
 <param name="checkFont" value="1"/>
 <param name="checkRestrict" value="1"/>
@@
 <wire x1="44.45" y1="39.0525" x2="44.45" y2="25.4" width="0.4064" layer="16"/>
 <wire x1="44.45" y1="25.4" x2="43.18" y2="24.13" width="0.4064" layer="16"/>
-<wire x1="43.18" y1="24.13" x2="38.735" y2="24.13" width="0.4064" layer="16"/>
+<wire x1="43.18" y1="24.13" x2="39.0525" y2="24.13" width="0.4064" layer="16"/>
 <via x="36.83" y="21.9075" extent="1-16" drill="0.6096" diameter="1.27"/>
-<wire x1="38.735" y1="24.13" x2="36.83" y2="21.9075" width="0.4064" layer="16"/>
+<wire x1="39.0525" y1="24.13" x2="36.83" y2="21.9075" width="0.4064" layer="16"/>
 <wire x1="36.83" y1="21.9075" x2="36.83" y2="18.7325" width="0.4064" layer="1"/>
 <wire x1="36.83" y1="18.7325" x2="39.37" y2="16.1925" width="0.4064" layer="1"/>
@@
 <wire x1="13.97" y1="65.405" x2="110.1725" y2="65.405" width="0.4064" layer="16"/>
 <wire x1="110.1725" y1="65.405" x2="111.4425" y2="64.135" width="0.4064" layer="16"/>
-<wire x1="111.4425" y1="64.135" x2="111.4425" y2="33.02" width="0.4064" layer="16"/>
-<wire x1="111.4425" y1="33.02" x2="116.84" y2="27.94" width="0.4064" layer="16"/>
+<wire x1="111.4425" y1="64.135" x2="111.4425" y2="33.3375" width="0.4064" layer="16"/>
+<wire x1="111.4425" y1="33.3375" x2="116.84" y2="27.94" width="0.4064" layer="16"/>
 <wire x1="116.84" y1="27.94" x2="118.11" y2="27.94" width="0.4064" layer="16"/>
 </signal>
@@
 <wire x1="109.5375" y1="77.7875" x2="104.4575" y2="82.8675" width="0.4064" layer="1"/>
 <wire x1="104.4575" y1="82.8675" x2="102.87" y2="82.8675" width="0.4064" layer="1"/>
-<wire x1="118.11" y1="50.8" x2="117.1575" y2="50.8" width="0.4064" layer="16"/>
-<wire x1="117.1575" y1="50.8" x2="112.395" y2="55.245" width="0.4064" layer="16"/>
-<wire x1="112.395" y1="55.245" x2="112.395" y2="64.135" width="0.4064" layer="16"/>
+<wire x1="118.11" y1="50.8" x2="116.205" y2="50.8" width="0.4064" layer="16"/>
+<wire x1="116.205" y1="50.8" x2="112.395" y2="54.61" width="0.4064" layer="16"/>
+<wire x1="112.395" y1="54.61" x2="112.395" y2="64.135" width="0.4064" layer="16"/>
 <wire x1="112.395" y1="64.135" x2="113.3475" y2="65.0875" width="0.4064" layer="16"/>
 <wire x1="113.3475" y1="65.0875" x2="113.3475" y2="76.835" width="0.4064" layer="16"/>

Commit message: 2016-02-10 17:30 (completed boards 2,6,7)
Parts:
- JP10: device pinhead:2X16 -> pinhead:2X18
- moved JP10 2.54 mm to (105.4, 6.99)
Connections:
- removed net /ENPPC: JP9.37
- new net /FP: JP10.34
- new net /IO: JP10.35
- new net /MEMOP: JP10.11
- new net /NP_FAULT: JP10.36
- new net /WR_FAULT: JP10.33
Changed lines of the file:
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@@
 <layer number="21" name="tPlace" color="7" fill="1" visible="no" active="yes"/>
 <layer number="22" name="bPlace" color="7" fill="1" visible="no" active="yes"/>
-<layer number="23" name="tOrigins" color="15" fill="1" visible="no" active="yes"/>
+<layer number="23" name="tOrigins" color="15" fill="1" visible="yes" active="yes"/>
 <layer number="24" name="bOrigins" color="15" fill="1" visible="no" active="yes"/>
 <layer number="25" name="tNames" color="7" fill="1" visible="no" active="yes"/>
@@
 <element name="JP3" library="pinhead" package="2X08" value="" x="6.0325" y="75.565" rot="R270"/>
 <element name="JP4" library="pinhead" package="2X08" value="" x="6.0325" y="24.765" rot="R270"/>
-<element name="JP10" library="pinhead" package="2X16" value="" x="107.95" y="6.985" rot="R180"/>
+<element name="JP10" library="pinhead" package="2X18" value="" x="105.41" y="6.985" rot="R180"/>
 <element name="JP9" library="pinhead" package="2X24" value="" x="48.26" y="6.985" rot="R180"/>
 <element name="JP5" library="pinhead" package="2X08" value="" x="6.0325" y="50.165" rot="R270"/>
@@
 <contactref element="JP9" pad="41"/>
 </signal>
-<signal name="/ENPPC">
-<contactref element="JP9" pad="37"/>
-</signal>
 <signal name="/ENMAR">
 <contactref element="JP9" pad="48"/>
@@
 <contactref element="JP9" pad="43"/>
 </signal>
+<signal name="/MEMOP">
+<contactref element="JP10" pad="11"/>
+</signal>
+<signal name="/WR_FAULT">
+<contactref element="JP10" pad="33"/>
+</signal>
+<signal name="/IO">
+<contactref element="JP10" pad="35"/>
+</signal>
+<signal name="/FP">
+<contactref element="JP10" pad="34"/>
+</signal>
+<signal name="/NP_FAULT">
+<contactref element="JP10" pad="36"/>
+</signal>
 </signals>

Commit message: Wed Feb 10 22:17:37 CET 2016 (completed boards 5,4)
Routing:
- net /CARRY3: track 116.2 -> 122.9 mm
- net /ALUSHR: track 134.8 -> 140.9 mm
- net /ENALU: track 188.9 -> 189.9 mm
Changed lines of the file:
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@@
 <layer number="21" name="tPlace" color="7" fill="1" visible="no" active="yes"/>
 <layer number="22" name="bPlace" color="7" fill="1" visible="no" active="yes"/>
-<layer number="23" name="tOrigins" color="15" fill="1" visible="yes" active="yes"/>
+<layer number="23" name="tOrigins" color="15" fill="1" visible="no" active="yes"/>
 <layer number="24" name="bOrigins" color="15" fill="1" visible="no" active="yes"/>
 <layer number="25" name="tNames" color="7" fill="1" visible="no" active="yes"/>
@@
 <layer number="97" name="Info" color="7" fill="1" visible="no" active="no"/>
 <layer number="98" name="Guide" color="6" fill="1" visible="no" active="no"/>
-<layer number="100" name="crosshair" color="7" fill="1" visible="yes" active="yes"/>
+<layer number="100" name="crosshair" color="7" fill="1" visible="no" active="yes"/>
 <layer number="121" name="tsilk" color="14" fill="1" visible="yes" active="yes"/>
-<layer number="122" name="bsilk" color="6" fill="1" visible="yes" active="yes"/>
+<layer number="122" name="bsilk" color="6" fill="1" visible="no" active="yes"/>
 </layers>
 <board>
@@
 <wire x1="0" y1="104.775" x2="-9.525" y2="104.775" width="0.2032" layer="100"/>
 <text x="126.6825" y="91.7575" size="3.81" layer="1" font="vector" ratio="15">#5</text>
+<wire x1="87.63" y1="5.08" x2="86.995" y2="4.445" width="0.2032" layer="121"/>
+<wire x1="85.725" y1="4.445" x2="86.995" y2="4.445" width="0.2032" layer="121"/>
+<wire x1="85.725" y1="4.445" x2="85.09" y2="5.08" width="0.2032" layer="121"/>
+<wire x1="85.09" y1="5.08" x2="84.455" y2="4.445" width="0.2032" layer="121"/>
+<wire x1="83.185" y1="4.445" x2="84.455" y2="4.445" width="0.2032" layer="121"/>
+<wire x1="83.185" y1="4.445" x2="82.55" y2="5.08" width="0.2032" layer="121"/>
+<wire x1="82.55" y1="8.89" x2="83.185" y2="9.525" width="0.2032" layer="121"/>
+<wire x1="84.455" y1="9.525" x2="83.185" y2="9.525" width="0.2032" layer="121"/>
+<wire x1="84.455" y1="9.525" x2="85.09" y2="8.89" width="0.2032" layer="121"/>
+<wire x1="85.09" y1="8.89" x2="85.725" y2="9.525" width="0.2032" layer="121"/>
+<wire x1="86.995" y1="9.525" x2="85.725" y2="9.525" width="0.2032" layer="121"/>
+<wire x1="86.995" y1="9.525" x2="87.63" y2="8.89" width="0.2032" layer="121"/>
+<wire x1="85.09" y1="5.08" x2="85.09" y2="8.89" width="0.2032" layer="121"/>
+<wire x1="82.55" y1="5.08" x2="82.55" y2="8.89" width="0.2032" layer="121"/>
 </plain>
 <attributes>
@@
 <wire x1="123.19" y1="73.9775" x2="121.92" y2="75.2475" width="0.4064" layer="1"/>
 <wire x1="121.92" y1="75.2475" x2="119.0625" y2="75.2475" width="0.4064" layer="1"/>
-<wire x1="76.2" y1="8.255" x2="84.7725" y2="8.255" width="0.4064" layer="1"/>
-<wire x1="84.7725" y1="8.255" x2="86.36" y2="9.8425" width="0.4064" layer="16"/>
-<wire x1="86.36" y1="9.8425" x2="120.3325" y2="9.8425" width="0.4064" layer="16"/>
-<wire x1="120.3325" y1="9.8425" x2="138.43" y2="27.94" width="0.4064" layer="16"/>
 <wire x1="138.43" y1="27.94" x2="138.43" y2="71.4375" width="0.4064" layer="16"/>
 <wire x1="138.43" y1="71.4375" x2="137.16" y2="72.7075" width="0.4064" layer="16"/>
 <wire x1="137.16" y1="72.7075" x2="135.255" y2="72.7075" width="0.4064" layer="16"/>
-<via x="84.7725" y="8.255" extent="1-16" drill="0.6096" diameter="1.27"/>
+<wire x1="76.2" y1="8.255" x2="80.645" y2="3.81" width="0.4064" layer="1"/>
+<via x="80.645" y="3.81" extent="1-16" drill="0.6096" diameter="1.27"/>
+<wire x1="80.645" y1="3.81" x2="86.36" y2="3.81" width="0.4064" layer="16"/>
+<wire x1="86.36" y1="3.81" x2="87.63" y2="5.08" width="0.4064" layer="16"/>
+<wire x1="87.63" y1="5.08" x2="87.63" y2="9.2075" width="0.4064" layer="16"/>
+<wire x1="87.63" y1="9.2075" x2="88.265" y2="9.8425" width="0.4064" layer="16"/>
+<wire x1="88.265" y1="9.8425" x2="120.3325" y2="9.8425" width="0.4064" layer="16"/>
+<wire x1="120.3325" y1="9.8425" x2="138.43" y2="27.94" width="0.4064" layer="16"/>
 </signal>
 <signal name="/ENALU">
@@
 <wire x1="29.21" y1="4.7625" x2="30.48" y2="3.4925" width="0.4064" layer="16"/>
 <wire x1="30.48" y1="3.4925" x2="77.7875" y2="3.4925" width="0.4064" layer="16"/>
-<wire x1="77.7875" y1="3.4925" x2="85.09" y2="10.795" width="0.4064" layer="16"/>
-<wire x1="85.09" y1="10.795" x2="120.015" y2="10.795" width="0.4064" layer="16"/>
-<wire x1="120.015" y1="10.795" x2="137.4775" y2="28.2575" width="0.4064" layer="16"/>
 <wire x1="137.4775" y1="28.2575" x2="137.4775" y2="53.975" width="0.4064" layer="16"/>
 <wire x1="137.4775" y1="53.975" x2="121.92" y2="69.5325" width="0.4064" layer="16"/>
@@
 <wire x1="121.92" y1="71.4375" x2="120.65" y2="72.7075" width="0.4064" layer="16"/>
 <wire x1="120.65" y1="72.7075" x2="119.0625" y2="72.7075" width="0.4064" layer="16"/>
+<wire x1="77.7875" y1="3.4925" x2="81.28" y2="6.985" width="0.4064" layer="16"/>
+<wire x1="81.28" y1="6.985" x2="84.455" y2="6.985" width="0.4064" layer="16"/>
+<wire x1="84.455" y1="6.985" x2="85.09" y2="7.62" width="0.4064" layer="16"/>
+<wire x1="85.09" y1="7.62" x2="85.09" y2="9.2075" width="0.4064" layer="16"/>
+<wire x1="85.09" y1="9.2075" x2="86.6775" y2="10.795" width="0.4064" layer="16"/>
+<wire x1="86.6775" y1="10.795" x2="120.015" y2="10.795" width="0.4064" layer="16"/>
+<wire x1="120.015" y1="10.795" x2="137.4775" y2="28.2575" width="0.4064" layer="16"/>
 </signal>
 <signal name="LBUS0">
@@
 <wire x1="36.83" y1="6.985" x2="36.83" y2="4.1275" width="0.4064" layer="1"/>
 <wire x1="36.83" y1="4.1275" x2="38.4175" y2="2.54" width="0.4064" layer="1"/>
-<wire x1="38.4175" y1="2.54" x2="81.5975" y2="2.54" width="0.4064" layer="1"/>
-<wire x1="86.995" y1="11.1125" x2="92.075" y2="16.1925" width="0.4064" layer="1"/>
-<wire x1="92.075" y1="16.1925" x2="105.7275" y2="16.1925" width="0.4064" layer="1"/>
-<wire x1="105.7275" y1="16.1925" x2="108.2675" y2="18.7325" width="0.4064" layer="1"/>
+<wire x1="38.4175" y1="2.54" x2="106.68" y2="2.54" width="0.4064" layer="1"/>
 <wire x1="108.2675" y1="18.7325" x2="108.2675" y2="43.18" width="0.4064" layer="16"/>
 <wire x1="108.2675" y1="43.18" x2="105.7275" y2="45.72" width="0.4064" layer="16"/>
 <wire x1="105.7275" y1="45.72" x2="102.87" y2="45.72" width="0.4064" layer="16"/>
 <via x="108.2675" y="18.7325" extent="1-16" drill="0.6096" diameter="1.27"/>
-<wire x1="81.5975" y1="2.54" x2="86.995" y2="7.9375" width="0.4064" layer="1"/>
-<wire x1="86.995" y1="7.9375" x2="86.995" y2="11.1125" width="0.4064" layer="1"/>
+<wire x1="106.68" y1="2.54" x2="107.95" y2="3.81" width="0.4064" layer="1"/>
+<wire x1="107.95" y1="3.81" x2="107.95" y2="18.415" width="0.4064" layer="1"/>
+<wire x1="107.95" y1="18.415" x2="108.2675" y2="18.7325" width="0.4064" layer="1"/>
 </signal>
 <signal name="N$1">
