File: eagle/1_cpu_mmu.sch (EAGLE design)
At the start: 47 parts, among them IC1 MT5C6408, IC10 74LS157N, IC11 74LS157N, IC12 74LS00N, IC13 74LS157N, IC14 74LS157N, IC17 74LS32N, IC19 74LS32N, IC2 MT5C6408, IC20 74LS02N, IC21 74LS374N, IC3 74LS27N, IC4 74LS20N, IC5 74LS08N, IC6 74LS245N, IC7 74LS245N, IC8 74LS32N, IC9 74LS157N

Commit message: MMU board updates 2016-03-16
Connections:
- net ABUS0: now also IC12A.I0
- net ABUS12: now also IC9A.1B
- net ABUS13: now also IC9A.2B
- net ABUS14: now also IC9A.3B
- net ABUS15: now also IC9A.4B
- net GND: no longer IC9A.1B, IC9A.2B, IC9A.3B, IC9A.4B
Other:
- moved on the sheet: C18, C20, IC17D, IC19A, IC19B, IC8P
