File: eagle/memory.sch (EAGLE design)
At the start: 47 parts, among them IC1 MT5C6408, IC10 74LS157N, IC11 74LS157N, IC12 74LS00N, IC13 74LS157N, IC14 74LS157N, IC17 74LS32N, IC19 74LS32N, IC2 MT5C6408, IC20 74LS02N, IC21 74LS374N, IC3 74LS27N, IC4 74LS20N, IC5 74LS08N, IC6 74LS245N, IC7 74LS245N, IC8 74LS32N, IC9 74LS157N

Commit message: MMU and Memory board updates, removed mem_ext board (obsolete)
Parts:
- removed C16, C17, C20: 100n, rcl:C-EU050-024X044
- removed C18: 10u, rcl:CPOL-EUE2.5-6
- removed GND1, GND2, VCC1, VCC2: (no value), pinhead:PINHD-2X2
- removed IC17, IC19: 74LS32N, 74xx-eu:74LS32N
- removed IC20: 74LS02N, 74xx-eu:74LS02N
- removed IC21: 74LS374N, 74xx-eu:74LS374N
- removed JP1, JP2, JP3, JP4: (no value), pinhead:PINHD-2X8
- removed JP10: (no value), pinhead:PINHD-2X18
- removed JP5: (no value), pinhead:PINHD-2X6
- added J1: DIN41612, 19inch:VG64B
- added RN1: 4k7, resistor-sil:G08R
- C15: value 100n -> 10u; device rcl:C-EU050-024X044 -> rcl:CPOL-EUE2.5-6
- IC1: value MT5C6408 -> 74LS245N; device dawid:MT5C6408 -> 74xx-eu:74LS245N
- IC10: value 74LS157N -> 74LS138N; device 74xx-eu:74LS157N -> 74xx-eu:74LS138N
- IC11, IC13, IC14: value 74LS157N -> 628512; device 74xx-eu:74LS157N -> hitachi_sram_hm628512a-series_rev1:HM628512A_DIL32
- IC12: value 74LS00N -> 628512; device 74xx-eu:74LS00N -> hitachi_sram_hm628512a-series_rev1:HM628512A_DIL32
- IC2: value MT5C6408 -> 74LS04N; device dawid:MT5C6408 -> 74xx-eu:74LS04N
- IC3: value 74LS27N -> 628512; device 74xx-eu:74LS27N -> hitachi_sram_hm628512a-series_rev1:HM628512A_DIL32
- IC4: value 74LS20N -> 628512; device 74xx-eu:74LS20N -> hitachi_sram_hm628512a-series_rev1:HM628512A_DIL32
- IC5: value 74LS08N -> 628512; device 74xx-eu:74LS08N -> hitachi_sram_hm628512a-series_rev1:HM628512A_DIL32
- IC6: value 74LS245N -> 628512; device 74xx-eu:74LS245N -> hitachi_sram_hm628512a-series_rev1:HM628512A_DIL32
- IC7: value 74LS245N -> AM29F010; device 74xx-eu:74LS245N -> am29-memory:AM29F010
- IC8: value 74LS32N -> 74LS139N; device 74xx-eu:74LS32N -> 74xx-eu:74LS139N
- IC9: value 74LS157N -> 74LS08N; device 74xx-eu:74LS157N -> 74xx-eu:74LS08N
Connections:
- removed net /ALUHI2MEM: JP10.25
- removed net /ALULO2MEM: JP10.29
- removed net /BUSIFCEN: JP10.5
- removed net /CNTSP: JP10.3
- removed net /ENABUS: JP10.22
- removed net /ENMEM: IC17A.I1, IC19D.I0, IC5B.I1, IC8B.I1, JP10.16
- removed net /ENPTAB: IC14A.4A, IC6A.DIR, IC7A.DIR, IC8B.O
- removed net /FI: JP10.32
- removed net /FIO: IC11A.3A, IC2G$1.DQ6, IC7A.A6
- removed net /FP: IC10A.!A!/B, IC11A.!A!/B, IC17C.I1, IC9A.!A!/B, JP10.34
- removed net /FPRESENT: IC12B.I0, IC2G$1.DQ8, IC7A.A8
- removed net /FS: IC14A.2B, IC21A.6D, IC3C.I2, JP10.30
- removed net /FWRITABLE: IC12D.I0, IC2G$1.DQ7, IC7A.A7
- removed net /INCPC: JP10.1
- removed net /LATCHFLAGS: JP10.12
- removed net /LDMEM: IC17B.I1, IC8A.I1, JP10.15
- removed net /LDPTAB: IC1G$1.!WE, IC2G$1.!WE, IC8A.O
- removed net /LOAD_IR: JP10.26
- removed net /MEM2ALUHI: JP10.27
- removed net /MEM2ALULO: JP10.31
- removed net /MEMOP: IC17C.I0, JP10.11
- removed net /NP_FAULT: IC12B.O, JP10.36
- removed net /PPREG: IC12C.I1, IC19D.I1, IC4B.O
- removed net /PTAB: IC12C.I0, IC13A.!A!/B, IC14A.!A!/B, IC4A.O, IC8A.I0, IC8B.I0, IC8C.I0, IC8D.I0
- removed net /RST: JP10.7
- removed net /WR_FAULT: IC12D.O, JP10.33
- removed net ALUBUS0: JP3.1
- removed net ALUBUS1: JP3.2
- removed net ALUBUS10: JP3.11
- removed net ALUBUS11: JP3.12
- removed net ALUBUS12: JP3.13
- removed net ALUBUS13: JP3.14
- removed net ALUBUS14: JP3.15
- removed net ALUBUS15: JP3.16
- removed net ALUBUS2: JP3.3
- removed net ALUBUS3: JP3.4
- removed net ALUBUS4: JP3.5
- removed net ALUBUS5: JP3.6
- removed net ALUBUS6: JP3.7
- removed net ALUBUS7: JP3.8
- removed net ALUBUS8: JP3.9
- removed net ALUBUS9: JP3.10
- removed net BUSCLKA: IC19C.I0, JP10.23
- removed net BUSCLKB: JP10.24
- removed net CLK0A: JP10.13
- removed net CLK0B: JP10.18
- removed net CLK0C: JP10.19
- removed net CLK0D: JP10.17
- removed net CLK1: JP10.10
- removed net FAULT: IC20C.I0, IC20C.I1, JP10.28
- removed net FC: JP10.2
- removed net FN: JP10.6
- removed net FV: JP10.8
- removed net FZ: JP10.4
- removed net IRQ0: JP1.2
- removed net IRQ1: JP1.4
- removed net IRQ2: JP1.6
- removed net IRQ3: JP1.8
- removed net IRQ4: JP1.10
- removed net IRQ5: JP1.12
- removed net IRQ6: JP1.14
- removed net IRQ7: JP1.16
- removed net MEMSEG: IC10A.2B, IC14A.1B, IC21A.5D, IC5A.I1, IC5D.I1, JP10.14
- removed net N$10: IC10A.2A, IC1G$1.DQ6, IC6A.A6
- removed net N$11: IC10A.3A, IC1G$1.DQ7, IC6A.A7
- removed net N$12: IC10A.4A, IC1G$1.DQ8, IC6A.A8
- removed net N$13: IC11A.1A, IC2G$1.DQ1, IC7A.A1
- removed net N$14: IC11A.2A, IC2G$1.DQ2, IC7A.A2
- removed net N$15: IC2G$1.DQ3, IC7A.A3
- removed net N$16: IC2G$1.DQ4, IC7A.A4
- removed net N$17: IC2G$1.DQ5, IC7A.A5
- removed net N$2: IC3B.O, IC4A.I1, IC4B.I1
- removed net N$20: IC17C.O, IC20A.I0
- removed net N$21: IC13A.1Y, IC1G$1.A0, IC2G$1.A0
- removed net N$22: IC13A.2Y, IC1G$1.A1, IC2G$1.A1
- removed net N$23: IC13A.3Y, IC1G$1.A2, IC2G$1.A2
- removed net N$24: IC13A.4Y, IC1G$1.A3, IC2G$1.A3
- removed net N$25: IC14A.1Y, IC1G$1.A4, IC2G$1.A4
- removed net N$26: IC14A.2Y, IC1G$1.A5, IC2G$1.A5
- removed net N$27: IC1G$1.CE2, IC7A.G, IC8C.O
- removed net N$28: IC2G$1.CE2, IC6A.G, IC8D.O
- removed net N$29: IC14A.4Y, IC1G$1.!OE, IC2G$1.!OE
- removed net N$30: IC12A.O, IC8C.I1
- removed net N$32: IC12C.O, IC17A.I0, IC17B.I0, IC20A.I1
- removed net N$33: IC12B.I1, IC20A.O, IC5B.I0
- removed net N$34: IC12D.I1, IC5B.O
- removed net N$36: IC5C.I1, IC5D.O
- removed net N$37: IC3C.O, IC4A.I2, IC4B.I2
- removed net N$38: IC4B.I3, IC5C.O
- removed net N$40: IC19C.I1, IC20C.O
- removed net N$41: IC19C.O, IC21A.CLK
- removed net N$42: IC19D.O, IC21A.OC
- removed net N$9: IC10A.1A, IC1G$1.DQ5, IC6A.A5
- removed net PROT: JP10.21
- removed net RBUS0: JP4.1
- removed net RBUS1: JP4.2
- removed net RBUS10: JP4.11
- removed net RBUS11: JP4.12
- removed net RBUS12: JP4.13
- removed net RBUS13: JP4.14
- removed net RBUS14: JP4.15
- removed net RBUS15: JP4.16
- removed net RBUS2: JP4.3
- removed net RBUS3: JP4.4
- removed net RBUS4: JP4.5
- removed net RBUS5: JP4.6
- removed net RBUS6: JP4.7
- removed net RBUS7: JP4.8
- removed net RBUS8: JP4.9
- removed net RBUS9: JP4.10
- removed net RST: JP10.9
- removed net SP_DIR: JP10.20
- new net /BANK0RAM: IC3.CE, IC9B.O
- new net /BANK1: IC10A.Y1, IC4.CE
- new net /BANK2: IC10A.Y2, IC5.CE
- new net /BANK3: IC10A.Y3, IC6.CE
- new net /BANK4: IC10A.Y4, IC11.CE
- new net /BANK5: IC10A.Y5, IC12.CE
- new net /BANK6: IC10A.Y6, IC13.CE
- new net /BANK7: IC10A.Y7, IC14.CE
- new net IDBUS0: IC11.I/O00, IC12.I/O00, IC13.I/O00, IC14.I/O00, IC1A.B1, IC3.I/O00, IC4.I/O00, IC5.I/O00, IC6.I/O00, IC7G$1.O0, RN1.2
- new net IDBUS1: IC11.I/O01, IC12.I/O01, IC13.I/O01, IC14.I/O01, IC1A.B2, IC3.I/O01, IC4.I/O01, IC5.I/O01, IC6.I/O01, IC7G$1.O1, RN1.3
- new net IDBUS2: IC11.I/O02, IC12.I/O02, IC13.I/O02, IC14.I/O02, IC1A.B3, IC3.I/O02, IC4.I/O02, IC5.I/O02, IC6.I/O02, IC7G$1.O2, RN1.4
- new net IDBUS3: IC11.I/O03, IC12.I/O03, IC13.I/O03, IC14.I/O03, IC1A.B4, IC3.I/O03, IC4.I/O03, IC5.I/O03, IC6.I/O03, IC7G$1.O3, RN1.5
- new net IDBUS4: IC11.I/O04, IC12.I/O04, IC13.I/O04, IC14.I/O04, IC1A.B5, IC3.I/O04, IC4.I/O04, IC5.I/O04, IC6.I/O04, IC7G$1.O4, RN1.6
- new net IDBUS5: IC11.I/O05, IC12.I/O05, IC13.I/O05, IC14.I/O05, IC1A.B6, IC3.I/O05, IC4.I/O05, IC5.I/O05, IC6.I/O05, IC7G$1.O5, RN1.7
- new net IDBUS6: IC11.I/O06, IC12.I/O06, IC13.I/O06, IC14.I/O06, IC1A.B7, IC3.I/O06, IC4.I/O06, IC5.I/O06, IC6.I/O06, IC7G$1.O6, RN1.8
- new net IDBUS7: IC11.I/O07, IC12.I/O07, IC13.I/O07, IC14.I/O07, IC1A.B8, IC3.I/O07, IC4.I/O07, IC5.I/O07, IC6.I/O07, IC7G$1.O7, RN1.9
- net +5V: now also C15.+, IC10A.G1, IC11.VCC, IC12.VCC, IC13.VCC, IC14.VCC, IC3.VCC, IC4.VCC, IC5.VCC, IC6.VCC, IC7G$1.WE/, J1.A31, J1.A32, J1.C31, J1.C32, RN1.1; no longer C15.1, C16.1, C17.1, C18.+, C20.1, IC11A.3B, IC11P.VCC, IC12P.VCC, IC13P.VCC, IC14P.VCC, IC17P.VCC, IC19P.VCC, IC20P.VCC, IC21A.7D, IC21A.8D, IC21P.VCC, IC3P.VCC, IC4P.VCC, IC5P.VCC, IC6P.VCC, VCC1.1, VCC1.2, VCC1.3, VCC1.4, VCC2.1, VCC2.2, VCC2.3, VCC2.4
- net /ENMEMX: now also IC11.OE, IC12.OE, IC13.OE, IC14.OE, IC1A.DIR, IC3.OE, IC4.OE, IC5.OE, IC6.OE, IC7G$1.!OE, J1.C22; no longer IC17A.O, JP5.11
- net /IO: now also IC2A.I, J1.C11; no longer IC11A.3Y, JP10.35
- net /LDMEMX: now also IC11.WE, IC12.WE, IC13.WE, IC14.WE, IC3.WE, IC4.WE, IC5.WE, IC6.WE, J1.A22; no longer IC17B.O, JP5.12
- net ABUS0: now also IC11.A0, IC12.A0, IC13.A0, IC14.A0, IC3.A0, IC4.A0, IC5.A0, IC6.A0, IC7G$1.A0, J1.C23; no longer IC12A.I1, IC8D.I1, JP2.1
- net ABUS1: now also IC11.A1, IC12.A1, IC13.A1, IC14.A1, IC3.A1, IC4.A1, IC5.A1, IC6.A1, IC7G$1.A1, J1.A23; no longer IC13A.1A, JP2.2
- net ABUS10: now also IC11.A10, IC12.A10, IC13.A10, IC14.A10, IC3.A10, IC4.A10, IC5.A10, IC6.A10, IC7G$1.A10, J1.C28; no longer IC3A.I2, JP2.11
- net ABUS11: now also IC11.A11, IC12.A11, IC13.A11, IC14.A11, IC3.A11, IC4.A11, IC5.A11, IC6.A11, IC7G$1.A11, J1.A28; no longer IC3B.I0, JP2.12
- net ABUS12: now also J1.C29; no longer IC13A.1B, IC21A.1D, IC3B.I1, JP2.13
- net ABUS13: now also J1.A29; no longer IC13A.2B, IC21A.2D, IC3B.I2, JP2.14
- net ABUS14: now also J1.C30; no longer IC13A.3B, IC21A.3D, IC3C.I0, JP2.15
- net ABUS15: now also J1.A30; no longer IC13A.4B, IC21A.4D, IC3C.I1, JP2.16
- net ABUS2: now also IC11.A2, IC12.A2, IC13.A2, IC14.A2, IC3.A2, IC4.A2, IC5.A2, IC6.A2, IC7G$1.A2, J1.C24; no longer IC13A.2A, JP2.3
- net ABUS3: now also IC11.A3, IC12.A3, IC13.A3, IC14.A3, IC3.A3, IC4.A3, IC5.A3, IC6.A3, IC7G$1.A3, J1.A24; no longer IC13A.3A, JP2.4
- net ABUS4: now also IC11.A4, IC12.A4, IC13.A4, IC14.A4, IC3.A4, IC4.A4, IC5.A4, IC6.A4, IC7G$1.A4, J1.C25; no longer IC13A.4A, JP2.5
- net ABUS5: now also IC11.A5, IC12.A5, IC13.A5, IC14.A5, IC3.A5, IC4.A5, IC5.A5, IC6.A5, IC7G$1.A5, J1.A25; no longer IC14A.1A, IC5D.I0, JP2.6
- net ABUS6: now also IC11.A6, IC12.A6, IC13.A6, IC14.A6, IC3.A6, IC4.A6, IC5.A6, IC6.A6, IC7G$1.A6, J1.C26; no longer IC14A.2A, JP2.7
- net ABUS7: now also IC11.A7, IC12.A7, IC13.A7, IC14.A7, IC3.A7, IC4.A7, IC5.A7, IC6.A7, IC7G$1.A7, J1.A26; no longer IC20B.I0, IC20B.I1, IC5A.I0, JP2.8
- net ABUS8: now also IC11.A8, IC12.A8, IC13.A8, IC14.A8, IC3.A8, IC4.A8, IC5.A8, IC6.A8, IC7G$1.A8, J1.C27; no longer IC3A.I0, JP2.9
- net ABUS9: now also IC11.A9, IC12.A9, IC13.A9, IC14.A9, IC3.A9, IC4.A9, IC5.A9, IC6.A9, IC7G$1.A9, J1.A27; no longer IC3A.I1, JP2.10
- net DBUS0: now also IC1A.A1, J1.C3; no longer IC21A.1Q, IC6A.B1, IC7A.B1, JP1.1
- net DBUS1: now also IC1A.A2, J1.C4; no longer IC21A.2Q, IC6A.B2, IC7A.B2, JP1.3
- net DBUS2: now also IC1A.A3, J1.C5; no longer IC21A.3Q, IC6A.B3, IC7A.B3, JP1.5
- net DBUS3: now also IC1A.A4, J1.C6; no longer IC21A.4Q, IC6A.B4, IC7A.B4, JP1.7
- net DBUS4: now also IC1A.A5, J1.C7; no longer IC21A.5Q, IC6A.B5, IC7A.B5, JP1.9
- net DBUS5: now also IC1A.A6, J1.C8; no longer IC21A.6Q, IC6A.B6, IC7A.B6, JP1.11
- net DBUS6: now also IC1A.A7, J1.C9; no longer IC21A.7Q, IC6A.B7, IC7A.B7, JP1.13
- net DBUS7: now also IC1A.A8, J1.C10; no longer IC21A.8Q, IC6A.B8, IC7A.B8, JP1.15
- net GND: now also C15.-, IC10A.G2A, IC10A.G2B, IC11.VSS, IC12.VSS, IC13.VSS, IC14.VSS, IC2B.I, IC2C.I, IC2D.I, IC2E.I, IC2F.I, IC3.VSS, IC4.VSS, IC5.VSS, IC6.VSS, IC8B.A, IC8B.B, IC8B.G, IC9C.I0, IC9C.I1, IC9D.I0, IC9D.I1, J1.A1, J1.A2, J1.C1, J1.C2; no longer C15.2, C16.2, C17.2, C18.-, C20.2, GND1.1, GND1.2, GND1.3, GND1.4, GND2.1, GND2.2, GND2.3, GND2.4, IC10A.1B, IC10A.3B, IC10A.4B, IC10A.G, IC11A.1B, IC11A.2B, IC11A.4A, IC11A.4B, IC11A.G, IC11P.GND, IC12P.GND, IC13A.G, IC13P.GND, IC14A.3A, IC14A.3B, IC14A.4B, IC14A.G, IC14P.GND, IC17D.I0, IC17D.I1, IC17P.GND, IC19A.I0, IC19A.I1, IC19B.I0, IC19B.I1, IC19P.GND, IC1G$1.!CE1, IC1G$1.A10, IC1G$1.A11, IC1G$1.A12, IC1G$1.A6, IC1G$1.A7, IC1G$1.A8, IC1G$1.A9, IC20D.I0, IC20D.I1, IC20P.GND, IC21P.GND, IC2G$1.!CE1, IC2G$1.A10, IC2G$1.A11, IC2G$1.A12, IC2G$1.A6, IC2G$1.A7, IC2G$1.A8, IC2G$1.A9, IC3P.GND, IC4P.GND, IC5P.GND, IC6P.GND, IC9A.1B, IC9A.2B, IC9A.3B, IC9A.4B, IC9A.G
- net N$1: now also IC1A.G, IC2A.O; no longer IC3A.O, IC4A.I0, IC4B.I0
- net N$3: now also IC10A.Y0, IC8A.G; no longer IC20B.O, IC5C.I0
- net N$4: now also IC8A.Y1, IC9A.I0; no longer IC4A.I3, IC5A.O
- net N$5: now also IC8A.Y2, IC9A.I1; no longer IC1G$1.DQ1, IC6A.A1, IC9A.1A
- net N$6: now also IC7G$1.!CE, IC8A.Y0; no longer IC1G$1.DQ2, IC6A.A2, IC9A.2A
- net N$7: now also IC8A.Y3, IC9B.I1; no longer IC1G$1.DQ3, IC6A.A3, IC9A.3A
- net N$8: now also IC9A.O, IC9B.I0; no longer IC1G$1.DQ4, IC6A.A4, IC9A.4A
- net PABUS12: now also IC11.A12, IC12.A12, IC13.A12, IC14.A12, IC3.A12, IC4.A12, IC5.A12, IC6.A12, IC7G$1.A12, J1.C15; no longer IC9A.1Y, JP5.1
- net PABUS13: now also IC11.A13, IC12.A13, IC13.A13, IC14.A13, IC3.A13, IC4.A13, IC5.A13, IC6.A13, IC7G$1.A13, J1.A15; no longer IC9A.2Y, JP5.2
- net PABUS14: now also IC11.A14, IC12.A14, IC13.A14, IC14.A14, IC3.A14, IC4.A14, IC5.A14, IC6.A14, IC7G$1.A14, J1.C16; no longer IC9A.3Y, JP5.3
- net PABUS15: now also IC11.A15, IC12.A15, IC13.A15, IC14.A15, IC3.A15, IC4.A15, IC5.A15, IC6.A15, IC7G$1.A15, J1.A16; no longer IC9A.4Y, JP5.4
- net PABUS16: now also IC11.A16, IC12.A16, IC13.A16, IC14.A16, IC3.A16, IC4.A16, IC5.A16, IC6.A16, IC7G$1.A16, J1.C17; no longer IC10A.1Y, JP5.5
- net PABUS17: now also IC11.A17, IC12.A17, IC13.A17, IC14.A17, IC3.A17, IC4.A17, IC5.A17, IC6.A17, IC8A.A, J1.A17; no longer IC10A.2Y, JP5.6
- net PABUS18: now also IC11.A18, IC12.A18, IC13.A18, IC14.A18, IC3.A18, IC4.A18, IC5.A18, IC6.A18, IC8A.B, J1.C18; no longer IC10A.3Y, JP5.7
- net PABUS19: now also IC10A.A, J1.A18; no longer IC10A.4Y, JP5.8
- net PABUS20: now also IC10A.B, J1.C19; no longer IC11A.1Y, JP5.9
- net PABUS21: now also IC10A.C, J1.A19; no longer IC11A.2Y, JP5.10
Other:
- note added: "MEM.1"
- note added: "Memory (ROM & RAM)"
- note removed: "(C) 2010-2014"
- note removed: "BOARD CONNECTORS"
- note removed: "CPU.1"
- note removed: "Memory Management Unit (MMU)"
- note removed: "fault preconditions"
