File: eagle/1_cpu_mmu.brd (EAGLE design)
At the start: 160 x 100 mm, 47 parts, among them IC1 MT5C6408, IC10 74LS157N, IC11 74LS157N, IC12 74LS00N, IC13 74LS157N, IC14 74LS157N, IC17 74LS32N, IC19 74LS32N, IC2 MT5C6408, IC20 74LS02N, IC21 74LS374N, IC3 74LS27N, IC4 74LS20N, IC5 74LS08N, IC6 74LS245N, IC7 74LS245N, IC8 74LS32N, IC9 74LS157N

Commit message: MMU board updates 2016-03-16
Parts:
- moved C13 115.7 mm to (15.2, 71.8), turned to 270 degrees
- moved C2 86.1 mm to (134.6, 69.2), turned to 90 degrees
- moved IC17 66.3 mm to (25.1, 29.8), turned to 180 degrees
- moved C12 62.4 mm to (59.4, 71.8), turned to 270 degrees
- moved IC12 61.5 mm to (52.7, 21.0), turned to 0 degrees
- moved C11 55.6 mm to (30.2, 55.6), turned to 270 degrees
- moved IC7 51.9 mm to (49.2, 88.9), turned to 180 degrees
- moved IC11 49.7 mm to (42.9, 54.3), turned to 0 degrees
- moved C3 47.2 mm to (104.5, 55.6), turned to 270 degrees
- moved C14 46.0 mm to (100.3, 16.5)
- moved C15 36.8 mm to (65.1, 16.5)
- moved IC19 36.5 mm to (34.0, 25.7)
- moved C1 36.2 mm to (66.0, 85.1), turned to 0 degrees
- moved IC20 33.1 mm to (21.6, 16.2)
- moved IC2 24.3 mm to (35.2, 70.5), turned to 0 degrees
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Connections:
- net ABUS0: now also IC12.1
- net ABUS12: now also IC9.3
- net ABUS13: now also IC9.6
- net ABUS14: now also IC9.10
- net ABUS15: now also IC9.13
- net GND: no longer IC9.10, IC9.13, IC9.3, IC9.6
Routing:
- net +5V: track 162.8 -> 407.8 mm
- net MEMSEG: track 147.2 -> 0.00 mm
- net DBUS6: track 60.1 -> 159.5 mm, vias 0 -> 2
- net DBUS5: track 50.3 -> 149.3 mm, vias 0 -> 2
- net DBUS4: track 48.0 -> 139.0 mm, vias 0 -> 1
- net ABUS15: track 101.2 -> 17.2 mm, vias 2 -> 0
- net DBUS7: track 76.9 -> 160.0 mm, vias 0 -> 1
- net ABUS13: track 107.6 -> 25.9 mm
- net ABUS14: track 99.5 -> 19.3 mm
- net ABUS12: track 112.7 -> 42.9 mm, vias 0 -> 1
- net PABUS20: track 68.6 -> 0.00 mm
- net /FS: track 65.1 -> 0.00 mm
- net N$8: track 83.7 -> 18.9 mm, vias 1 -> 0
- net /FIO: track 79.4 -> 18.9 mm
- net PABUS21: track 57.6 -> 0.00 mm
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
Commit message: MMU board updates 2016-03-24
Parts:
- moved C5 69.7 mm to (54.3, 56.5), turned to 270 degrees
- moved C4 59.0 mm to (27.9, 56.5), turned to 270 degrees
- moved C15 47.6 mm to (112.1, 23.8), turned to 270 degrees
- moved IC19 40.5 mm to (73.0, 14.9), turned to 0 degrees
- moved C14 38.1 mm to (62.2, 16.2), turned to 270 degrees
- moved IC14 36.1 mm to (40.3, 54.3)
- moved IC13 35.7 mm to (66.7, 54.3)
- moved C10 34.9 mm to (62.5, 30.8), turned to 270 degrees
- moved C8 29.0 mm to (36.8, 30.8), turned to 270 degrees
- moved C6 28.1 mm to (13.0, 30.8), turned to 270 degrees
- moved IC11 27.6 mm to (15.2, 54.3)
- moved C11 22.0 mm to (8.89, 61.3), turned to 0 degrees
- moved IC5 17.5 mm to (47.6, 14.9), turned to 0 degrees
- moved C7 16.4 mm to (13.0, 16.2), turned to 270 degrees
- moved C9 14.4 mm to (36.8, 17.1), turned to 270 degrees
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Routing:
- net +5V: track 407.8 -> 786.9 mm
- net MEMSEG: track 0.00 -> 217.3 mm, vias 0 -> 3
- net ABUS14: track 19.3 -> 202.3 mm, vias 0 -> 3
- net ABUS15: track 17.2 -> 187.8 mm, vias 0 -> 1
- net ABUS12: track 42.9 -> 207.6 mm, vias 1 -> 2
- net ABUS7: track 0.00 -> 149.7 mm, vias 0 -> 1
- net ABUS13: track 25.9 -> 171.0 mm, vias 0 -> 1
- net N$28: track 0.00 -> 138.1 mm, vias 0 -> 3
- net /ENMEMX: track 0.00 -> 134.0 mm, vias 0 -> 1
- net PABUS20: track 0.00 -> 132.1 mm
- net /LDMEMX: track 0.00 -> 129.3 mm, vias 0 -> 1
- net PABUS21: track 0.00 -> 127.0 mm
- net ABUS5: track 0.00 -> 122.3 mm, vias 0 -> 1
- net ABUS0: track 0.00 -> 116.4 mm, vias 0 -> 1
- net ABUS6: track 0.00 -> 112.9 mm, vias 0 -> 1
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
Commit message: MMU board updates 2016-04-13
Parts:
- moved C10 5.12 mm to (60.0, 35.2), turned to 90 degrees
- moved C16 4.55 mm to (80.6, 60.6), turned to 90 degrees
- moved C9 2.93 mm to (36.2, 14.3)
- moved C12 2.86 mm to (62.5, 78.1)
- moved C8 1.31 mm to (36.5, 29.5)
- moved C4 0.95 mm to (27.9, 55.6)
Routing:
- net /FS: track 45.3 -> 193.8 mm, vias 0 -> 2
- net /FP: track 27.8 -> 167.9 mm, vias 0 -> 1
- net /ENMEM: track 0.00 -> 123.7 mm, vias 0 -> 3
- net /MEMOP: track 0.00 -> 122.8 mm, vias 0 -> 1
- net /IO: track 0.00 -> 111.8 mm, vias 0 -> 1
- net /LDMEM: track 0.00 -> 107.2 mm, vias 0 -> 1
- net /ENPTAB: track 112.1 -> 202.9 mm, vias 1 -> 3
- net /PTAB: track 49.1 -> 138.0 mm, vias 0 -> 1
- net FAULT: track 0.00 -> 82.4 mm, vias 0 -> 1
- net /PPREG: track 0.00 -> 75.7 mm, vias 0 -> 2
- net N$32: track 0.00 -> 72.2 mm, vias 0 -> 1
- net N$41: track 0.00 -> 67.7 mm
- net GND: track 45.7 -> 110.5 mm
- net /WR_FAULT: track 0.00 -> 64.6 mm, vias 0 -> 2
- net N$4: track 0.00 -> 63.3 mm, vias 0 -> 1
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- added copper zone on layer 1, net GND
- added copper zone on layer 16, net GND

Commit message: MMU board completed
Parts:
- moved C13 0.64 mm to (18.7, 80.0)
- moved C15 0.64 mm to (111.4, 23.8)
- moved C2 0.32 mm to (134.9, 69.2)
Routing:
- net GND: track 110.5 -> 132.3 mm, vias 0 -> 1
- net /PPREG: track 75.7 -> 80.8 mm
- net +5V: track 799.3 -> 802.9 mm
- net ABUS0: track 131.1 -> 132.9 mm
- net /LDMEM: track 107.2 -> 108.2 mm
- net ABUS7: track 155.0 -> 156.0 mm
Other:
- board text added: "10u"
- board text added: "74LS00N"
- board text added: "74LS02N"
- board text added: "74LS08N"
- board text added: "74LS157N"
- board text added: "74LS20N"
- board text added: "74LS245N"
- board text added: "74LS27N"
- board text added: "74LS32N"
- board text added: "74LS374N"
- board text added: "GND1"
- board text added: "GND2"
- board text added: "IC1"
- board text added: "IC10"
- board text added: "IC11"
- board text added: "IC12"
- board text added: "IC13"
- board text added: "IC14"
- board text added: "IC17"
- board text added: "IC19"
- board text added: "IC2"
- board text added: "IC20"
- board text added: "IC21"
- board text added: "IC3"
- board text added: "IC4"
- board text added: "IC5"
- board text added: "IC6"
- board text added: "IC7"
- board text added: "IC8"
- board text added: "IC9"
- board text added: "JP1"
- board text added: "JP10"
- board text added: "JP2"
- board text added: "JP3"
- board text added: "JP4"
- board text added: "JP5"
- board text added: "MT5C6408"
- board text added: "VCC1"
- board text added: "VCC2"
